Commit message: 不要なフレームを削除

File: urdf/crane_x7_d435.xacro (robot description, xacro)
@@ -3,5 +3,4 @@
   <xacro:macro name="d435"
       params="parent
-              use_gazebo
               *origin">
     <joint name="camera_joint" type="fixed">
@@ -38,36 +37,4 @@
     </joint>
     <link name="camera_link"/>
-    <xacro:if value="$(arg use_gazebo)">
-      <joint name="camera_depth_frame_joint" type="fixed">
-        <origin xyz="0 0 0" rpy="0 0 0"/>
-        <parent link="camera_link"/>
-        <child  link="camera_depth_frame"/>
-      </joint>
-      <link name="camera_depth_frame"/>
-      <joint name="camera_depth_optical_frame_joint" type="fixed">
-        <origin xyz="0 0 0" rpy="${radians(-90)} 0 ${radians(-90)}"/>
-        <parent link="camera_depth_frame"/>
-        <child  link="camera_depth_optical_frame"/>
-      </joint>
-      <link name="camera_depth_optical_frame"/>
-      <joint name="camera_color_frame_joint" type="fixed">
-        <origin xyz="0 0.015 0" rpy="0 0 0"/>
-        <parent link="camera_link"/>
-        <child  link="camera_color_frame"/>
-      </joint>
-      <link name="camera_color_frame"/>
-      <joint name="camera_color_optical_frame_joint" type="fixed">
-        <origin xyz="0 0 0" rpy="${radians(-90)} 0 ${radians(-90)}"/>
-        <parent link="camera_color_frame"/>
-        <child  link="camera_color_optical_frame"/>
-      </joint>
-      <link name="camera_color_optical_frame"/>
-      <joint name="camera_aligned_depth_to_color_frame_joint" type="fixed">
-        <origin xyz="0 0.015 0" rpy="0 0 0"/>
-        <parent link="camera_link"/>
-        <child  link="camera_aligned_depth_to_color_frame"/>
-      </joint>
-      <link name="camera_aligned_depth_to_color_frame"/>
-    </xacro:if>
   </xacro:macro>
 </robot>

Commit message: D435のメッシュ更新

File: urdf/crane_x7_d435.xacro (robot description, xacro)
@@ -11,16 +11,13 @@
     <link name="camera_base">
       <inertial>
-        <mass value="0.6"/>
+        <mass value="0.072"/>
         <origin xyz="0 0 0" rpy="0 0 0"/>
         <inertia ixx="1e-3" ixy="0.0" ixz="0.0" iyy="1e-3" iyz="0.0" izz="1e-3"/>
       </inertial>
       <visual>
-        <origin xyz="${0.025/2} 0 0" rpy="0 0 0"/>
+        <origin xyz="0.025 0 0" rpy="${radians(90)} 0 ${radians(90)}"/>
         <geometry>
-          <box size="0.025 0.09 0.025"/>
+          <mesh filename="package://realsense2_description/meshes/d435.dae" />
         </geometry>
-        <material name="yellow">
-          <color rgba="1 1 0 1" />
-        </material>
       </visual>
       <collision>
