Commit message: Fix gripper mimic joint control

File: urdf/crane_x7.gazebo_ros2_control.xacro (robot description, xacro)
@@ -11,4 +11,5 @@
             name_joint_7
             name_joint_gripper_finger_a
+            name_joint_gripper_finger_b
             joint_1_lower_limit
             joint_1_upper_limit
@@ -104,4 +105,12 @@
         <state_interface name="effort"/>
       </joint>
+    <joint name="${name_joint_gripper_finger_b}">
+      <param name="mimic">${name_joint_gripper_finger_a}</param>
+      <param name="multiplier">1</param>
+      <command_interface name="position"/>
+      <state_interface name="position"/>
+      <state_interface name="velocity"/>
+      <state_interface name="effort"/>
+    </joint>
     </ros2_control>
   </xacro:macro>

File: urdf/crane_x7.urdf.xacro (robot description, xacro)
@@ -241,4 +241,5 @@
       name_joint_7="${NAME_JOINT_7}"
       name_joint_gripper_finger_a="${NAME_JOINT_GRIPPER_FINGER_A}"
+      name_joint_gripper_finger_b="${NAME_JOINT_GRIPPER_FINGER_B}"
       joint_1_lower_limit="${JOINT_1_LOWER_LIMIT}"
       joint_1_upper_limit="${JOINT_1_UPPER_LIMIT}"

Commit message: スタイル修正

File: urdf/crane_x7.gazebo_ros2_control.xacro (robot description, xacro)
@@ -29,4 +29,5 @@
             joint_hand_upper_limit
             ">
+    <ros2_control name="${name}" type="system">
       <hardware>
         <plugin>gz_ros2_control/GazeboSimSystem</plugin>
@@ -104,12 +105,12 @@
         <state_interface name="effort"/>
       </joint>
-    <joint name="${name_joint_gripper_finger_b}">
-      <param name="mimic">${name_joint_gripper_finger_a}</param>
-      <param name="multiplier">1</param>
-      <command_interface name="position"/>
-      <state_interface name="position"/>
-      <state_interface name="velocity"/>
-      <state_interface name="effort"/>
-    </joint>
+      <joint name="${name_joint_gripper_finger_b}">
+        <param name="mimic">${name_joint_gripper_finger_a}</param>
+        <param name="multiplier">1</param>
+        <command_interface name="position"/>
+        <state_interface name="position"/>
+        <state_interface name="velocity"/>
+        <state_interface name="effort"/>
+      </joint>
     </ros2_control>
   </xacro:macro>
