Commit message: D435追加(Gazebo未対応)

File: urdf/crane_x7.gazebo.xacro (robot description, xacro)
@@ -50,4 +50,5 @@
             config_package
             config_file_path
+            use_d435
             ">
     <gazebo>
@@ -117,4 +118,71 @@
       <xacro:material_gazebo_red/>
     </gazebo>
+    <xacro:if value="$(arg use_d435)">
+      <gazebo reference="camera_link">
+        <sensor type="depth" name="camera1">
+          <update_rate>30.0</update_rate>
+          <visualize>false</visualize>
+          <camera>
+            <horizontal_fov>${radians(69.4)}</horizontal_fov>
+            <image>
+              <width>640</width>
+              <height>480</height>
+              <format>B8G8R8</format>
+            </image>
+            <depth_camera>
+            </depth_camera>
+            <clip>
+              <near>0.02</near>
+              <far>300</far>
+            </clip>
+            <noise>
+              <type>gaussian</type>
+              <mean>0.0</mean>
+              <stddev>0.007</stddev>
+            </noise>
+          </camera>
+          <plugin name="camera_controller" filename="libgazebo_ros_camera.so">
+            <ros>
+              <namespace>demo_cam</namespace>
+              <remapping>depth_camera/image_raw:=fake_cam_color/image_raw</remapping>
+              <remapping>depth_camera/camera_info:=fake_cam_color/camera_info</remapping>
+              <remapping>depth_camera/points:=depth_camera/depth/color/points</remapping>
+            </ros>
+            <camera_name>depth_camera</camera_name>
+            <min_depth>0.105</min_depth>
+            <max_depth>10.0</max_depth>
+          </plugin>
+        </sensor>
+      </gazebo>
+      <!--
+      <gazebo reference="camera_aligned_depth_to_color_frame">
+        <sensor type="depth" name="camera2">
+          <update_rate>30.0</update_rate>
+          <camera name="color_camera">
+            <horizontal_fov>${radians(69.4)}</horizontal_fov>
+            <image>
+              <width>640</width>
+              <height>480</height>
+              <format>B8G8R8</format>
+            </image>
+            <clip>
+              <near>0.02</near>
+              <far>300</far>
+            </clip>
+          </camera>
+          <plugin name="camera_plugin" filename="libgazebo_ros_openni_kinect.so">
+            <baseline>0.2</baseline>
+            <alwaysOn>true</alwaysOn>
+            <updateRate>0.0</updateRate>
+            <cameraName>camera</cameraName>
+            <imageTopicName>color/image_raw</imageTopicName>
+            <depthImageTopicName>aligned_depth_to_color/image_raw</depthImageTopicName>
+            <cameraInfoTopicName>color/camera_info</cameraInfoTopicName>
+            <depthImageCameraInfoTopicName>aligned_depth_to_color/camera_info</depthImageCameraInfoTopicName>
+          </plugin>
+        </sensor>
+      </gazebo>
+      -->
+    </xacro:if>
   </xacro:macro>
 </robot>

File: urdf/crane_x7.urdf.xacro (robot description, xacro)
@@ -8,8 +8,10 @@
   <!-- Include the Crane X7 generator macro -->
   <xacro:include filename="$(find crane_x7_description)/urdf/crane_x7.xacro"/>
+  <xacro:include filename="$(find crane_x7_description)/urdf/crane_x7_d435.xacro"/>
   <xacro:include filename="$(find crane_x7_description)/urdf/crane_x7.ros2_control.xacro"/>
   <xacro:include filename="$(find crane_x7_description)/urdf/crane_x7.gazebo.xacro"/>
   <xacro:include filename="$(find crane_x7_description)/urdf/crane_x7.gazebo_ros2_control.xacro"/>
   <xacro:arg name="use_gazebo" default="false" />
+  <xacro:arg name="use_d435" default="false" />
   <xacro:arg name="port_name" default="/dev/ttyUSB0" />
   <xacro:arg name="baudrate" default="3000000" />
@@ -166,5 +168,7 @@
     joint_7_upper_limit="${JOINT_7_UPPER_LIMIT}"
     joint_hand_lower_limit="${JOINT_HAND_LOWER_LIMIT}"
-    joint_hand_upper_limit="${JOINT_HAND_UPPER_LIMIT}">
+    joint_hand_upper_limit="${JOINT_HAND_UPPER_LIMIT}"
+    use_d435="$(arg use_d435)"
+    use_gazebo="$(arg use_gazebo)">
     <origin xyz="0 0 0"/>
   </xacro:crane_x7>
@@ -226,4 +230,5 @@
       config_package="$(arg gz_control_config_package)"
       config_file_path="$(arg gz_control_config_file_path)"
+      use_d435="$(arg use_d435)"
       />
     <xacro:crane_x7_gazebo_ros2_control_settings

File: urdf/crane_x7.xacro (robot description, xacro)
@@ -91,4 +91,6 @@
               joint_hand_lower_limit
               joint_hand_upper_limit
+              use_d435
+              use_gazebo
               *origin">
     <!-- Mounting plate
@@ -162,4 +164,12 @@
       <origin xyz="0 0 ${MOUNTING_PLATE_THICKNESS}" rpy="0 0 0"/>
     </xacro:crane_x7_arm>
+    <!-- RealSense D435 -->
+    <xacro:if value="$(arg use_d435)">
+      <xacro:d435
+          parent="${name_link_7}"
+          use_gazebo="$(arg use_gazebo)">
+        <origin xyz="0.0 0.0445 0.009" rpy="${radians(-90)} ${radians(-90)} 0"/>
+      </xacro:d435>
+    </xacro:if>
     <!-- End effector -->
     <xacro:crane_x7_wide_two_finger_gripper
