Commit message: 残りのマクロのパラメータも削除

File: urdf/crane_x7.gazebo.xacro (robot description, xacro)
@@ -25,89 +25,67 @@
     </visual>
   </xacro:macro>
-  <xacro:macro name="gazebo_robot_settings"
-    params="name_link_mounting_plate
-            name_link_base
-            name_link_1
-            name_link_2
-            name_link_3
-            name_link_4
-            name_link_5
-            name_link_6
-            name_link_cover_2_l
-            name_link_cover_2_r
-            name_link_cover_4_l
-            name_link_cover_4_r
-            name_link_logo_symbol_l
-            name_link_logo_symbol_r
-            name_link_logo_text_l
-            name_link_logo_text_r
-            name_link_gripper_base
-            name_link_gripper_finger_a
-            name_link_gripper_finger_b
-            config_package
-            config_file_path
-            ">
+  <xacro:macro name="gazebo_robot_settings">
     <gazebo>
       <plugin filename="libgz_ros2_control-system.so" name="gz_ros2_control::GazeboSimROS2ControlPlugin">
-        <parameters>$(find ${config_package})/${config_file_path}</parameters>
+        <parameters>$(find ${GZ_CONTROL_CONFIG_PACKAGE})/${GZ_CONTROL_CONFIG_FILE_PATH}</parameters>
       </plugin>
     </gazebo>
-    <gazebo reference="${name_link_mounting_plate}">
+    <gazebo reference="${NAME_LINK_MOUNTING_PLATE}">
       <xacro:material_gazebo_black/>
     </gazebo>
-    <gazebo reference="${name_link_base}">
+    <gazebo reference="${NAME_LINK_BASE}">
       <xacro:material_gazebo_red/>
     </gazebo>
-    <gazebo reference="${name_link_1}">
+    <gazebo reference="${NAME_LINK_1}">
       <xacro:material_gazebo_white/>
     </gazebo>
-    <gazebo reference="${name_link_2}">
+    <gazebo reference="${NAME_LINK_2}">
       <xacro:material_gazebo_white/>
     </gazebo>
-    <gazebo reference="${name_link_3}">
+    <gazebo reference="${NAME_LINK_3}">
       <xacro:material_gazebo_white/>
     </gazebo>
-    <gazebo reference="${name_link_4}">
+    <gazebo reference="${NAME_LINK_4}">
       <xacro:material_gazebo_white/>
     </gazebo>
-    <gazebo reference="${name_link_5}">
+    <gazebo reference="${NAME_LINK_5}">
       <xacro:material_gazebo_white/>
     </gazebo>
-    <gazebo reference="${name_link_6}">
+    <gazebo reference="${NAME_LINK_6}">
       <xacro:material_gazebo_white/>
     </gazebo>
-    <gazebo reference="${name_link_cover_2_l}">
+    <gazebo reference="${NAME_LINK_COVER_2_L}">
       <xacro:material_gazebo_red/>
     </gazebo>
-    <gazebo reference="${name_link_cover_2_r}">
+    <gazebo reference="${NAME_LINK_COVER_2_R}">
       <xacro:material_gazebo_red/>
     </gazebo>
-    <gazebo reference="${name_link_cover_4_l}">
+    <gazebo reference="${NAME_LINK_COVER_4_L}">
       <xacro:material_gazebo_red/>
     </gazebo>
-    <gazebo reference="${name_link_cover_4_r}">
+    <gazebo reference="${NAME_LINK_COVER_4_R}">
       <xacro:material_gazebo_red/>
     </gazebo>
-    <gazebo reference="${name_link_logo_symbol_l}">
+    <gazebo reference="${NAME_LINK_LOGO_SYMBOL_L}">
       <xacro:material_gazebo_red/>
     </gazebo>
-    <gazebo reference="${name_link_logo_symbol_r}">
+    <gazebo reference="${NAME_LINK_LOGO_SYMBOL_R}">
       <xacro:material_gazebo_red/>
     </gazebo>
-    <gazebo reference="${name_link_logo_text_l}">
+    <gazebo reference="${NAME_LINK_LOGO_TEXT_L}">
       <xacro:material_gazebo_black/>
     </gazebo>
-    <gazebo reference="${name_link_logo_text_r}">
+    <gazebo reference="${NAME_LINK_LOGO_TEXT_R}">
       <xacro:material_gazebo_black/>
     </gazebo>
-    <gazebo reference="${name_link_gripper_base}">
+    <gazebo reference="${NAME_LINK_GRIPPER_BASE}">
       <xacro:material_gazebo_red/>
     </gazebo>
-    <gazebo reference="${name_link_gripper_finger_a}">
+    <gazebo reference="${NAME_LINK_GRIPPER_FINGER_A}">
       <mu1>0.8</mu1>
       <mu2>0.8</mu2>
       <xacro:material_gazebo_red/>
     </gazebo>
-    <gazebo reference="${name_link_gripper_finger_b}">
+    <gazebo reference="${NAME_LINK_GRIPPER_FINGER_B}">
       <mu1>0.8</mu1>
       <mu2>0.8</mu2>

File: urdf/crane_x7.gazebo_ros2_control.xacro (robot description, xacro)
@@ -1,40 +1,13 @@
 <?xml version="1.0"?>
 <robot xmlns:xacro="http://www.ros.org/wiki/xacro">
-  <xacro:macro name="crane_x7_gazebo_ros2_control_settings"
-    params="name
-            name_joint_1
-            name_joint_2
-            name_joint_3
-            name_joint_4
-            name_joint_5
-            name_joint_6
-            name_joint_7
-            name_joint_gripper_finger_a
-            name_joint_gripper_finger_b
-            joint_1_lower_limit
-            joint_1_upper_limit
-            joint_2_lower_limit
-            joint_2_upper_limit
-            joint_3_lower_limit
-            joint_3_upper_limit
-            joint_4_lower_limit
-            joint_4_upper_limit
-            joint_5_lower_limit
-            joint_5_upper_limit
-            joint_6_lower_limit
-            joint_6_upper_limit
-            joint_7_lower_limit
-            joint_7_upper_limit
-            joint_hand_lower_limit
-            joint_hand_upper_limit
-            ">
-    <ros2_control name="${name}" type="system">
+  <xacro:macro name="crane_x7_gazebo_ros2_control_settings">
+    <ros2_control name="crane_x7" type="system">
       <hardware>
         <plugin>gz_ros2_control/GazeboSimSystem</plugin>
       </hardware>
-      <joint name="${name_joint_1}">
+      <joint name="${NAME_JOINT_1}">
         <command_interface name="position">
-          <param name="min">${joint_1_lower_limit}</param>
-          <param name="max">${joint_1_upper_limit}</param>
+          <param name="min">${JOINT_1_LOWER_LIMIT}</param>
+          <param name="max">${JOINT_1_UPPER_LIMIT}</param>
         </command_interface>
         <state_interface name="position"/>
@@ -42,8 +15,8 @@
         <state_interface name="effort"/>
       </joint>
-      <joint name="${name_joint_2}">
+      <joint name="${NAME_JOINT_2}">
         <command_interface name="position">
-          <param name="min">${joint_2_lower_limit}</param>
-          <param name="max">${joint_2_upper_limit}</param>
+          <param name="min">${JOINT_2_LOWER_LIMIT}</param>
+          <param name="max">${JOINT_2_UPPER_LIMIT}</param>
         </command_interface>
         <state_interface name="position"/>
@@ -51,8 +24,8 @@
         <state_interface name="effort"/>
       </joint>
-      <joint name="${name_joint_3}">
+      <joint name="${NAME_JOINT_3}">
         <command_interface name="position">
-          <param name="min">${joint_3_lower_limit}</param>
-          <param name="max">${joint_3_upper_limit}</param>
+          <param name="min">${JOINT_3_LOWER_LIMIT}</param>
+          <param name="max">${JOINT_3_UPPER_LIMIT}</param>
         </command_interface>
         <state_interface name="position"/>
@@ -60,8 +33,8 @@
         <state_interface name="effort"/>
       </joint>
-      <joint name="${name_joint_4}">
+      <joint name="${NAME_JOINT_4}">
         <command_interface name="position">
-          <param name="min">${joint_4_lower_limit}</param>
-          <param name="max">${joint_4_upper_limit}</param>
+          <param name="min">${JOINT_4_LOWER_LIMIT}</param>
+          <param name="max">${JOINT_4_UPPER_LIMIT}</param>
         </command_interface>
         <state_interface name="position"/>
@@ -69,8 +42,8 @@
         <state_interface name="effort"/>
       </joint>
-      <joint name="${name_joint_5}">
+      <joint name="${NAME_JOINT_5}">
         <command_interface name="position">
-          <param name="min">${joint_5_lower_limit}</param>
-          <param name="max">${joint_5_upper_limit}</param>
+          <param name="min">${JOINT_5_LOWER_LIMIT}</param>
+          <param name="max">${JOINT_5_UPPER_LIMIT}</param>
         </command_interface>
         <state_interface name="position"/>
@@ -78,8 +51,8 @@
         <state_interface name="effort"/>
       </joint>
-      <joint name="${name_joint_6}">
+      <joint name="${NAME_JOINT_6}">
         <command_interface name="position">
-          <param name="min">${joint_6_lower_limit}</param>
-          <param name="max">${joint_6_upper_limit}</param>
+          <param name="min">${JOINT_6_LOWER_LIMIT}</param>
+          <param name="max">${JOINT_6_UPPER_LIMIT}</param>
         </command_interface>
         <state_interface name="position"/>
@@ -87,8 +60,8 @@
         <state_interface name="effort"/>
       </joint>
-      <joint name="${name_joint_7}">
+      <joint name="${NAME_JOINT_7}">
         <command_interface name="position">
-          <param name="min">${joint_7_lower_limit}</param>
-          <param name="max">${joint_7_upper_limit}</param>
+          <param name="min">${JOINT_7_LOWER_LIMIT}</param>
+          <param name="max">${JOINT_7_UPPER_LIMIT}</param>
         </command_interface>
         <state_interface name="position"/>
@@ -96,8 +69,8 @@
         <state_interface name="effort"/>
       </joint>
-      <joint name="${name_joint_gripper_finger_a}">
+      <joint name="${NAME_JOINT_GRIPPER_FINGER_A}">
         <command_interface name="position">
-          <param name="min">${joint_hand_lower_limit}</param>
-          <param name="max">${joint_hand_upper_limit}</param>
+          <param name="min">${JOINT_HAND_LOWER_LIMIT}</param>
+          <param name="max">${JOINT_HAND_UPPER_LIMIT}</param>
         </command_interface>
         <state_interface name="position"/>
@@ -105,6 +78,6 @@
         <state_interface name="effort"/>
       </joint>
-      <joint name="${name_joint_gripper_finger_b}">
-        <param name="mimic">${name_joint_gripper_finger_a}</param>
+      <joint name="${NAME_JOINT_GRIPPER_FINGER_B}">
+        <param name="mimic">${NAME_JOINT_GRIPPER_FINGER_A}</param>
         <param name="multiplier">1</param>
         <state_interface name="position"/>

File: urdf/crane_x7.ros2_control.xacro (robot description, xacro)
@@ -1,55 +1,23 @@
 <?xml version="1.0"?>
 <robot xmlns:xacro="http://www.ros.org/wiki/xacro">
-  <xacro:macro name="crane_x7_ros2_control_settings"
-    params="name
-            name_joint_1
-            name_joint_2
-            name_joint_3
-            name_joint_4
-            name_joint_5
-            name_joint_6
-            name_joint_7
-            name_joint_gripper_finger_a
-            joint_1_lower_limit
-            joint_1_upper_limit
-            joint_2_lower_limit
-            joint_2_upper_limit
-            joint_3_lower_limit
-            joint_3_upper_limit
-            joint_4_lower_limit
-            joint_4_upper_limit
-            joint_5_lower_limit
-            joint_5_upper_limit
-            joint_6_lower_limit
-            joint_6_upper_limit
-            joint_7_lower_limit
-            joint_7_upper_limit
-            joint_hand_lower_limit
-            joint_hand_upper_limit
-            port_name
-            baudrate
-            timeout_seconds
-            manipulator_config_file_path
-            manipulator_links_file_path
-            use_mock_components
-            ">
-    <ros2_control name="${name}" type="system">
+  <xacro:macro name="crane_x7_ros2_control_settings">
+    <ros2_control name="crane_x7" type="system">
       <hardware>
-        <xacro:if value="${use_mock_components}">
+        <xacro:if value="${USE_MOCK_COMPONENTS}">
           <plugin>mock_components/GenericSystem</plugin>
         </xacro:if>
-        <xacro:unless value="${use_mock_components}">
+        <xacro:unless value="${USE_MOCK_COMPONENTS}">
           <plugin>crane_x7_hardware/CraneX7Hardware</plugin>
-          <param name="port_name">${port_name}</param>
-          <param name="baudrate">${baudrate}</param>
-          <param name="timeout_seconds">${timeout_seconds}</param>
-          <param name="manipulator_config_file_path">${manipulator_config_file_path}</param>
-          <param name="manipulator_links_file_path">${manipulator_links_file_path}</param>
+          <param name="port_name">${PORT_NAME}</param>
+          <param name="baudrate">${BAUDRATE}</param>
+          <param name="timeout_seconds">${TIMEOUT_SECONDS}</param>
+          <param name="manipulator_config_file_path">${MANIPULATOR_CONFIG_FILE_PATH}</param>
+          <param name="manipulator_links_file_path">${MANIPULATOR_LINKS_FILE_PATH}</param>
         </xacro:unless>
       </hardware>
-      <joint name="${name_joint_1}">
+      <joint name="${NAME_JOINT_1}">
         <command_interface name="position">
-          <param name="min">${joint_1_lower_limit}</param>
-          <param name="max">${joint_1_upper_limit}</param>
+          <param name="min">${JOINT_1_LOWER_LIMIT}</param>
+          <param name="max">${JOINT_1_UPPER_LIMIT}</param>
         </command_interface>
         <state_interface name="position"/>
@@ -58,8 +26,8 @@
         <param name="current_to_effort">2.20</param>
       </joint>
-      <joint name="${name_joint_2}">
+      <joint name="${NAME_JOINT_2}">
         <command_interface name="position">
-          <param name="min">${joint_2_lower_limit}</param>
-          <param name="max">${joint_2_upper_limit}</param>
+          <param name="min">${JOINT_2_LOWER_LIMIT}</param>
+          <param name="max">${JOINT_2_UPPER_LIMIT}</param>
         </command_interface>
         <state_interface name="position"/>
@@ -68,8 +36,8 @@
         <param name="current_to_effort">3.60</param>
       </joint>
-      <joint name="${name_joint_3}">
+      <joint name="${NAME_JOINT_3}">
         <command_interface name="position">
-          <param name="min">${joint_3_lower_limit}</param>
-          <param name="max">${joint_3_upper_limit}</param>
+          <param name="min">${JOINT_3_LOWER_LIMIT}</param>
+          <param name="max">${JOINT_3_UPPER_LIMIT}</param>
         </command_interface>
         <state_interface name="position"/>
@@ -78,8 +46,8 @@
         <param name="current_to_effort">2.20</param>
       </joint>
-      <joint name="${name_joint_4}">
+      <joint name="${NAME_JOINT_4}">
         <command_interface name="position">
-          <param name="min">${joint_4_lower_limit}</param>
-          <param name="max">${joint_4_upper_limit}</param>
+          <param name="min">${JOINT_4_LOWER_LIMIT}</param>
+          <param name="max">${JOINT_4_UPPER_LIMIT}</param>
         </command_interface>
         <state_interface name="position"/>
@@ -88,8 +56,8 @@
         <param name="current_to_effort">2.20</param>
       </joint>
-      <joint name="${name_joint_5}">
+      <joint name="${NAME_JOINT_5}">
         <command_interface name="position">
-          <param name="min">${joint_5_lower_limit}</param>
-          <param name="max">${joint_5_upper_limit}</param>
+          <param name="min">${JOINT_5_LOWER_LIMIT}</param>
+          <param name="max">${JOINT_5_UPPER_LIMIT}</param>
         </command_interface>
         <state_interface name="position"/>
@@ -98,8 +66,8 @@
         <param name="current_to_effort">2.20</param>
       </joint>
-      <joint name="${name_joint_6}">
+      <joint name="${NAME_JOINT_6}">
         <command_interface name="position">
-          <param name="min">${joint_6_lower_limit}</param>
-          <param name="max">${joint_6_upper_limit}</param>
+          <param name="min">${JOINT_6_LOWER_LIMIT}</param>
+          <param name="max">${JOINT_6_UPPER_LIMIT}</param>
         </command_interface>
         <state_interface name="position"/>
@@ -108,8 +76,8 @@
         <param name="current_to_effort">2.20</param>
       </joint>
-      <joint name="${name_joint_7}">
+      <joint name="${NAME_JOINT_7}">
         <command_interface name="position">
-          <param name="min">${joint_7_lower_limit}</param>
-          <param name="max">${joint_7_upper_limit}</param>
+          <param name="min">${JOINT_7_LOWER_LIMIT}</param>
+          <param name="max">${JOINT_7_UPPER_LIMIT}</param>
         </command_interface>
         <state_interface name="position"/>
@@ -118,8 +86,8 @@
         <param name="current_to_effort">2.20</param>
       </joint>
-      <joint name="${name_joint_gripper_finger_a}">
+      <joint name="${NAME_JOINT_GRIPPER_FINGER_A}">
         <command_interface name="position">
-          <param name="min">${joint_hand_lower_limit}</param>
-          <param name="max">${joint_hand_upper_limit}</param>
+          <param name="min">${JOINT_HAND_LOWER_LIMIT}</param>
+          <param name="max">${JOINT_HAND_UPPER_LIMIT}</param>
         </command_interface>
         <state_interface name="position"/>

File: urdf/crane_x7.urdf.xacro (robot description, xacro)
@@ -110,89 +110,9 @@
   </xacro:crane_x7>
   <xacro:unless value="$(arg use_gazebo)">
-    <xacro:crane_x7_ros2_control_settings
-      name="crane_x7"
-      name_joint_1="${NAME_JOINT_1}"
-      name_joint_2="${NAME_JOINT_2}"
-      name_joint_3="${NAME_JOINT_3}"
-      name_joint_4="${NAME_JOINT_4}"
-      name_joint_5="${NAME_JOINT_5}"
-      name_joint_6="${NAME_JOINT_6}"
-      name_joint_7="${NAME_JOINT_7}"
-      name_joint_gripper_finger_a="${NAME_JOINT_GRIPPER_FINGER_A}"
-      joint_1_lower_limit="${JOINT_1_LOWER_LIMIT}"
-      joint_1_upper_limit="${JOINT_1_UPPER_LIMIT}"
-      joint_2_lower_limit="${JOINT_2_LOWER_LIMIT}"
-      joint_2_upper_limit="${JOINT_2_UPPER_LIMIT}"
-      joint_3_lower_limit="${JOINT_3_LOWER_LIMIT}"
-      joint_3_upper_limit="${JOINT_3_UPPER_LIMIT}"
-      joint_4_lower_limit="${JOINT_4_LOWER_LIMIT}"
-      joint_4_upper_limit="${JOINT_4_UPPER_LIMIT}"
-      joint_5_lower_limit="${JOINT_5_LOWER_LIMIT}"
-      joint_5_upper_limit="${JOINT_5_UPPER_LIMIT}"
-      joint_6_lower_limit="${JOINT_6_LOWER_LIMIT}"
-      joint_6_upper_limit="${JOINT_6_UPPER_LIMIT}"
-      joint_7_lower_limit="${JOINT_7_LOWER_LIMIT}"
-      joint_7_upper_limit="${JOINT_7_UPPER_LIMIT}"
-      joint_hand_lower_limit="${JOINT_HAND_LOWER_LIMIT}"
-      joint_hand_upper_limit="${JOINT_HAND_UPPER_LIMIT}"
-      port_name="$(arg port_name)"
-      baudrate="$(arg baudrate)"
-      timeout_seconds="$(arg timeout_seconds)"
-      manipulator_config_file_path="$(arg manipulator_config_file_path)"
-      manipulator_links_file_path="$(arg manipulator_links_file_path)"
-      use_mock_components="$(arg use_mock_components)"
-      />
+    <xacro:crane_x7_ros2_control_settings/>
   </xacro:unless>
   <xacro:if value="$(arg use_gazebo)">
-    <xacro:gazebo_robot_settings
-      name_link_mounting_plate="${NAME_LINK_MOUNTING_PLATE}"
-      name_link_base="${NAME_LINK_BASE}"
-      name_link_1="${NAME_LINK_1}"
-      name_link_2="${NAME_LINK_2}"
-      name_link_3="${NAME_LINK_3}"
-      name_link_4="${NAME_LINK_4}"
-      name_link_5="${NAME_LINK_5}"
-      name_link_6="${NAME_LINK_6}"
-      name_link_cover_2_l="${NAME_LINK_COVER_2_L}"
-      name_link_cover_2_r="${NAME_LINK_COVER_2_R}"
-      name_link_cover_4_l="${NAME_LINK_COVER_4_L}"
-      name_link_cover_4_r="${NAME_LINK_COVER_4_R}"
-      name_link_logo_symbol_l="${NAME_LINK_LOGO_SYMBOL_L}"
-      name_link_logo_symbol_r="${NAME_LINK_LOGO_SYMBOL_R}"
-      name_link_logo_text_l="${NAME_LINK_LOGO_TEXT_L}"
-      name_link_logo_text_r="${NAME_LINK_LOGO_TEXT_R}"
-      name_link_gripper_base="${NAME_LINK_GRIPPER_BASE}"
-      name_link_gripper_finger_a="${NAME_LINK_GRIPPER_FINGER_A}"
-      name_link_gripper_finger_b="${NAME_LINK_GRIPPER_FINGER_B}"
-      config_package="$(arg gz_control_config_package)"
-      config_file_path="$(arg gz_control_config_file_path)"
-      />
-    <xacro:crane_x7_gazebo_ros2_control_settings
-      name="crane_x7"
-      name_joint_1="${NAME_JOINT_1}"
-      name_joint_2="${NAME_JOINT_2}"
-      name_joint_3="${NAME_JOINT_3}"
-      name_joint_4="${NAME_JOINT_4}"
-      name_joint_5="${NAME_JOINT_5}"
-      name_joint_6="${NAME_JOINT_6}"
-      name_joint_7="${NAME_JOINT_7}"
-      name_joint_gripper_finger_a="${NAME_JOINT_GRIPPER_FINGER_A}"
-      name_joint_gripper_finger_b="${NAME_JOINT_GRIPPER_FINGER_B}"
-      joint_1_lower_limit="${JOINT_1_LOWER_LIMIT}"
-      joint_1_upper_limit="${JOINT_1_UPPER_LIMIT}"
-      joint_2_lower_limit="${JOINT_2_LOWER_LIMIT}"
-      joint_2_upper_limit="${JOINT_2_UPPER_LIMIT}"
-      joint_3_lower_limit="${JOINT_3_LOWER_LIMIT}"
-      joint_3_upper_limit="${JOINT_3_UPPER_LIMIT}"
-      joint_4_lower_limit="${JOINT_4_LOWER_LIMIT}"
-      joint_4_upper_limit="${JOINT_4_UPPER_LIMIT}"
-      joint_5_lower_limit="${JOINT_5_LOWER_LIMIT}"
-      joint_5_upper_limit="${JOINT_5_UPPER_LIMIT}"
-      joint_6_lower_limit="${JOINT_6_LOWER_LIMIT}"
-      joint_6_upper_limit="${JOINT_6_UPPER_LIMIT}"
-      joint_7_lower_limit="${JOINT_7_LOWER_LIMIT}"
-      joint_7_upper_limit="${JOINT_7_UPPER_LIMIT}"
-      joint_hand_lower_limit="${JOINT_HAND_LOWER_LIMIT}"
-      joint_hand_upper_limit="${JOINT_HAND_UPPER_LIMIT}" />
+    <xacro:gazebo_robot_settings/>
+    <xacro:crane_x7_gazebo_ros2_control_settings/>
   </xacro:if>
 </robot>
