Commit message: リンクとジョイントのpropertyを廃止

File: urdf/crane_x7.gazebo.xacro (robot description, xacro)
@@ -26,24 +26,5 @@
   </xacro:macro>
   <xacro:macro name="gazebo_robot_settings"
-    params="name_link_mounting_plate
-            name_link_base
-            name_link_1
-            name_link_2
-            name_link_3
-            name_link_4
-            name_link_5
-            name_link_6
-            name_link_cover_2_l
-            name_link_cover_2_r
-            name_link_cover_4_l
-            name_link_cover_4_r
-            name_link_logo_symbol_l
-            name_link_logo_symbol_r
-            name_link_logo_text_l
-            name_link_logo_text_r
-            name_link_gripper_base
-            name_link_gripper_finger_a
-            name_link_gripper_finger_b
-            config_package
+    params="config_package
             config_file_path
             ">
@@ -53,61 +34,61 @@
       </plugin>
     </gazebo>
-    <gazebo reference="${name_link_mounting_plate}">
+    <gazebo reference="crane_x7_mounting_plate_link">
       <xacro:material_gazebo_black/>
     </gazebo>
-    <gazebo reference="${name_link_base}">
+    <gazebo reference="crane_x7_shoulder_fixed_part_link">
       <xacro:material_gazebo_red/>
     </gazebo>
-    <gazebo reference="${name_link_1}">
+    <gazebo reference="crane_x7_shoulder_revolute_part_link">
       <xacro:material_gazebo_white/>
     </gazebo>
-    <gazebo reference="${name_link_2}">
+    <gazebo reference="crane_x7_upper_arm_fixed_part_link">
       <xacro:material_gazebo_white/>
     </gazebo>
-    <gazebo reference="${name_link_3}">
+    <gazebo reference="crane_x7_upper_arm_revolute_part_link">
       <xacro:material_gazebo_white/>
     </gazebo>
-    <gazebo reference="${name_link_4}">
+    <gazebo reference="crane_x7_lower_arm_fixed_part_link">
       <xacro:material_gazebo_white/>
     </gazebo>
-    <gazebo reference="${name_link_5}">
+    <gazebo reference="crane_x7_lower_arm_revolute_part_link">
       <xacro:material_gazebo_white/>
     </gazebo>
-    <gazebo reference="${name_link_6}">
+    <gazebo reference="crane_x7_wrist_link">
       <xacro:material_gazebo_white/>
     </gazebo>
-    <gazebo reference="${name_link_cover_2_l}">
+    <gazebo reference="crane_x7_upper_arm_fixed_part_joint_cover_l_link">
       <xacro:material_gazebo_red/>
     </gazebo>
-    <gazebo reference="${name_link_cover_2_r}">
+    <gazebo reference="crane_x7_upper_arm_fixed_part_joint_cover_r_link">
       <xacro:material_gazebo_red/>
     </gazebo>
-    <gazebo reference="${name_link_cover_4_l}">
+    <gazebo reference="crane_x7_lower_arm_fixed_part_joint_cover_l_link">
       <xacro:material_gazebo_red/>
     </gazebo>
-    <gazebo reference="${name_link_cover_4_r}">
+    <gazebo reference="crane_x7_lower_arm_fixed_part_joint_cover_r_link">
       <xacro:material_gazebo_red/>
     </gazebo>
-    <gazebo reference="${name_link_logo_symbol_l}">
+    <gazebo reference="crane_x7_lower_arm_revolute_part_logo_symbol_l_link">
       <xacro:material_gazebo_red/>
     </gazebo>
-    <gazebo reference="${name_link_logo_symbol_r}">
+    <gazebo reference="crane_x7_lower_arm_revolute_part_logo_symbol_r_link">
       <xacro:material_gazebo_red/>
     </gazebo>
-    <gazebo reference="${name_link_logo_text_l}">
+    <gazebo reference="crane_x7_lower_arm_revolute_part_logo_text_l_link">
       <xacro:material_gazebo_black/>
     </gazebo>
-    <gazebo reference="${name_link_logo_text_r}">
+    <gazebo reference="crane_x7_lower_arm_revolute_part_logo_text_r_link">
       <xacro:material_gazebo_black/>
     </gazebo>
-    <gazebo reference="${name_link_gripper_base}">
+    <gazebo reference="crane_x7_gripper_base_link">
       <xacro:material_gazebo_red/>
     </gazebo>
-    <gazebo reference="${name_link_gripper_finger_a}">
+    <gazebo reference="crane_x7_gripper_finger_a_link">
       <mu1>0.8</mu1>
       <mu2>0.8</mu2>
       <xacro:material_gazebo_red/>
     </gazebo>
-    <gazebo reference="${name_link_gripper_finger_b}">
+    <gazebo reference="crane_x7_gripper_finger_b_link">
       <mu1>0.8</mu1>
       <mu2>0.8</mu2>

File: urdf/crane_x7.gazebo_ros2_control.xacro (robot description, xacro)
@@ -3,13 +3,4 @@
   <xacro:macro name="crane_x7_gazebo_ros2_control_settings"
     params="name
-            name_joint_1
-            name_joint_2
-            name_joint_3
-            name_joint_4
-            name_joint_5
-            name_joint_6
-            name_joint_7
-            name_joint_gripper_finger_a
-            name_joint_gripper_finger_b
             joint_1_lower_limit
             joint_1_upper_limit
@@ -33,5 +24,5 @@
         <plugin>gz_ros2_control/GazeboSimSystem</plugin>
       </hardware>
-      <joint name="${name_joint_1}">
+      <joint name="crane_x7_shoulder_fixed_part_pan_joint">
         <command_interface name="position">
           <param name="min">${joint_1_lower_limit}</param>
@@ -42,5 +33,5 @@
         <state_interface name="effort"/>
       </joint>
-      <joint name="${name_joint_2}">
+      <joint name="crane_x7_shoulder_revolute_part_tilt_joint">
         <command_interface name="position">
           <param name="min">${joint_2_lower_limit}</param>
@@ -51,5 +42,5 @@
         <state_interface name="effort"/>
       </joint>
-      <joint name="${name_joint_3}">
+      <joint name="crane_x7_upper_arm_revolute_part_twist_joint">
         <command_interface name="position">
           <param name="min">${joint_3_lower_limit}</param>
@@ -60,5 +51,5 @@
         <state_interface name="effort"/>
       </joint>
-      <joint name="${name_joint_4}">
+      <joint name="crane_x7_upper_arm_revolute_part_rotate_joint">
         <command_interface name="position">
           <param name="min">${joint_4_lower_limit}</param>
@@ -69,5 +60,5 @@
         <state_interface name="effort"/>
       </joint>
-      <joint name="${name_joint_5}">
+      <joint name="crane_x7_lower_arm_fixed_part_joint">
         <command_interface name="position">
           <param name="min">${joint_5_lower_limit}</param>
@@ -78,5 +69,5 @@
         <state_interface name="effort"/>
       </joint>
-      <joint name="${name_joint_6}">
+      <joint name="crane_x7_lower_arm_revolute_part_joint">
         <command_interface name="position">
           <param name="min">${joint_6_lower_limit}</param>
@@ -87,5 +78,5 @@
         <state_interface name="effort"/>
       </joint>
-      <joint name="${name_joint_7}">
+      <joint name="crane_x7_wrist_joint">
         <command_interface name="position">
           <param name="min">${joint_7_lower_limit}</param>
@@ -96,5 +87,5 @@
         <state_interface name="effort"/>
       </joint>
-      <joint name="${name_joint_gripper_finger_a}">
+      <joint name="crane_x7_gripper_finger_a_joint">
         <command_interface name="position">
           <param name="min">${joint_hand_lower_limit}</param>
@@ -105,6 +96,6 @@
         <state_interface name="effort"/>
       </joint>
-      <joint name="${name_joint_gripper_finger_b}">
-        <param name="mimic">${name_joint_gripper_finger_a}</param>
+      <joint name="crane_x7_gripper_finger_b_joint">
+        <param name="mimic">crane_x7_gripper_finger_a_joint</param>
         <param name="multiplier">1</param>
         <state_interface name="position"/>

File: urdf/crane_x7.ros2_control.xacro (robot description, xacro)
@@ -3,12 +3,4 @@
   <xacro:macro name="crane_x7_ros2_control_settings"
     params="name
-            name_joint_1
-            name_joint_2
-            name_joint_3
-            name_joint_4
-            name_joint_5
-            name_joint_6
-            name_joint_7
-            name_joint_gripper_finger_a
             joint_1_lower_limit
             joint_1_upper_limit
@@ -48,5 +40,5 @@
         </xacro:unless>
       </hardware>
-      <joint name="${name_joint_1}">
+      <joint name="crane_x7_shoulder_fixed_part_pan_joint">
         <command_interface name="position">
           <param name="min">${joint_1_lower_limit}</param>
@@ -58,5 +50,5 @@
         <param name="current_to_effort">2.20</param>
       </joint>
-      <joint name="${name_joint_2}">
+      <joint name="crane_x7_shoulder_revolute_part_tilt_joint">
         <command_interface name="position">
           <param name="min">${joint_2_lower_limit}</param>
@@ -68,5 +60,5 @@
         <param name="current_to_effort">3.60</param>
       </joint>
-      <joint name="${name_joint_3}">
+      <joint name="crane_x7_upper_arm_revolute_part_twist_joint">
         <command_interface name="position">
           <param name="min">${joint_3_lower_limit}</param>
@@ -78,5 +70,5 @@
         <param name="current_to_effort">2.20</param>
       </joint>
-      <joint name="${name_joint_4}">
+      <joint name="crane_x7_upper_arm_revolute_part_rotate_joint">
         <command_interface name="position">
           <param name="min">${joint_4_lower_limit}</param>
@@ -88,5 +80,5 @@
         <param name="current_to_effort">2.20</param>
       </joint>
-      <joint name="${name_joint_5}">
+      <joint name="crane_x7_lower_arm_fixed_part_joint">
         <command_interface name="position">
           <param name="min">${joint_5_lower_limit}</param>
@@ -98,5 +90,5 @@
         <param name="current_to_effort">2.20</param>
       </joint>
-      <joint name="${name_joint_6}">
+      <joint name="crane_x7_lower_arm_revolute_part_joint">
         <command_interface name="position">
           <param name="min">${joint_6_lower_limit}</param>
@@ -108,5 +100,5 @@
         <param name="current_to_effort">2.20</param>
       </joint>
-      <joint name="${name_joint_7}">
+      <joint name="crane_x7_wrist_joint">
         <command_interface name="position">
           <param name="min">${joint_7_lower_limit}</param>
@@ -118,5 +110,5 @@
         <param name="current_to_effort">2.20</param>
       </joint>
-      <joint name="${name_joint_gripper_finger_a}">
+      <joint name="crane_x7_gripper_finger_a_joint">
         <command_interface name="position">
           <param name="min">${joint_hand_lower_limit}</param>

File: urdf/crane_x7.urdf.xacro (robot description, xacro)
@@ -30,43 +30,4 @@
   </joint>
   <xacro:property name="M_PI" value="3.14159"/>
-  <xacro:property name="NAME_LINK_MOUNTING_PLATE" value="crane_x7_mounting_plate_link"/>
-  <xacro:property name="NAME_LINK_BASE" value="crane_x7_shoulder_fixed_part_link"/>
-  <xacro:property name="NAME_LINK_1" value="crane_x7_shoulder_revolute_part_link"/>
-  <xacro:property name="NAME_LINK_2" value="crane_x7_upper_arm_fixed_part_link"/>
-  <xacro:property name="NAME_LINK_3" value="crane_x7_upper_arm_revolute_part_link"/>
-  <xacro:property name="NAME_LINK_4" value="crane_x7_lower_arm_fixed_part_link"/>
-  <xacro:property name="NAME_LINK_5" value="crane_x7_lower_arm_revolute_part_link"/>
-  <xacro:property name="NAME_LINK_6" value="crane_x7_wrist_link"/>
-  <xacro:property name="NAME_LINK_7" value="crane_x7_gripper_base_link"/>
-  <xacro:property name="NAME_LINK_COVER_2_L" value="crane_x7_upper_arm_fixed_part_joint_cover_l_link"/>
-  <xacro:property name="NAME_LINK_COVER_2_R" value="crane_x7_upper_arm_fixed_part_joint_cover_r_link"/>
-  <xacro:property name="NAME_LINK_COVER_4_L" value="crane_x7_lower_arm_fixed_part_joint_cover_l_link"/>
-  <xacro:property name="NAME_LINK_COVER_4_R" value="crane_x7_lower_arm_fixed_part_joint_cover_r_link"/>
-  <xacro:property name="NAME_LINK_LOGO_SYMBOL_L" value="crane_x7_lower_arm_revolute_part_logo_symbol_l_link"/>
-  <xacro:property name="NAME_LINK_LOGO_SYMBOL_R" value="crane_x7_lower_arm_revolute_part_logo_symbol_r_link"/>
-  <xacro:property name="NAME_LINK_LOGO_TEXT_L" value="crane_x7_lower_arm_revolute_part_logo_text_l_link"/>
-  <xacro:property name="NAME_LINK_LOGO_TEXT_R" value="crane_x7_lower_arm_revolute_part_logo_text_r_link"/>
-  <xacro:property name="NAME_LINK_GRIPPER_BASE" value="crane_x7_gripper_base_link"/>
-  <xacro:property name="NAME_LINK_GRIPPER_FINGER_A" value="crane_x7_gripper_finger_a_link"/>
-  <xacro:property name="NAME_LINK_GRIPPER_FINGER_B" value="crane_x7_gripper_finger_b_link"/>
-  <xacro:property name="NAME_JOINT_MOUNTING_PLATE" value="crane_x7_mounting_plate_joint"/>
-  <xacro:property name="NAME_JOINT_BASE" value="crane_x7_shoulder_fixed_part_mount_joint"/>
-  <xacro:property name="NAME_JOINT_1" value="crane_x7_shoulder_fixed_part_pan_joint"/>
-  <xacro:property name="NAME_JOINT_2" value="crane_x7_shoulder_revolute_part_tilt_joint"/>
-  <xacro:property name="NAME_JOINT_3" value="crane_x7_upper_arm_revolute_part_twist_joint"/>
-  <xacro:property name="NAME_JOINT_4" value="crane_x7_upper_arm_revolute_part_rotate_joint"/>
-  <xacro:property name="NAME_JOINT_5" value="crane_x7_lower_arm_fixed_part_joint"/>
-  <xacro:property name="NAME_JOINT_6" value="crane_x7_lower_arm_revolute_part_joint"/>
-  <xacro:property name="NAME_JOINT_7" value="crane_x7_wrist_joint"/>
-  <xacro:property name="NAME_JOINT_COVER_2_L" value="crane_x7_upper_arm_fixed_part_joint_cover_l_joint"/>
-  <xacro:property name="NAME_JOINT_COVER_2_R" value="crane_x7_upper_arm_fixed_part_joint_cover_r_joint"/>
-  <xacro:property name="NAME_JOINT_COVER_4_L" value="crane_x7_lower_arm_fixed_part_joint_cover_l_joint"/>
-  <xacro:property name="NAME_JOINT_COVER_4_R" value="crane_x7_lower_arm_fixed_part_joint_cover_r_joint"/>
-  <xacro:property name="NAME_JOINT_LOGO_SYMBOL_L" value="crane_x7_lower_arm_revolute_part_logo_symbol_l_joint"/>
-  <xacro:property name="NAME_JOINT_LOGO_SYMBOL_R" value="crane_x7_lower_arm_revolute_part_logo_symbol_r_joint"/>
-  <xacro:property name="NAME_JOINT_LOGO_TEXT_L" value="crane_x7_lower_arm_revolute_part_logo_text_l_joint"/>
-  <xacro:property name="NAME_JOINT_LOGO_TEXT_R" value="crane_x7_lower_arm_revolute_part_logo_text_r_joint"/>
-  <xacro:property name="NAME_JOINT_GRIPPER_FINGER_A" value="crane_x7_gripper_finger_a_joint"/>
-  <xacro:property name="NAME_JOINT_GRIPPER_FINGER_B" value="crane_x7_gripper_finger_b_joint"/>
   <xacro:property name="COLOR_LINK_BASE" value="red"/>
   <xacro:property name="COLOR_LINK_1" value="white"/>
@@ -105,43 +66,4 @@
   <xacro:crane_x7
     parent="base_link"
-    name_link_mounting_plate="${NAME_LINK_MOUNTING_PLATE}"
-    name_link_base="${NAME_LINK_BASE}"
-    name_link_1="${NAME_LINK_1}"
-    name_link_2="${NAME_LINK_2}"
-    name_link_3="${NAME_LINK_3}"
-    name_link_4="${NAME_LINK_4}"
-    name_link_5="${NAME_LINK_5}"
-    name_link_6="${NAME_LINK_6}"
-    name_link_7="${NAME_LINK_7}"
-    name_link_cover_2_l="${NAME_LINK_COVER_2_L}"
-    name_link_cover_2_r="${NAME_LINK_COVER_2_R}"
-    name_link_cover_4_l="${NAME_LINK_COVER_4_L}"
-    name_link_cover_4_r="${NAME_LINK_COVER_4_R}"
-    name_link_logo_symbol_l="${NAME_LINK_LOGO_SYMBOL_L}"
-    name_link_logo_symbol_r="${NAME_LINK_LOGO_SYMBOL_R}"
-    name_link_logo_text_l="${NAME_LINK_LOGO_TEXT_L}"
-    name_link_logo_text_r="${NAME_LINK_LOGO_TEXT_R}"
-    name_link_gripper_base="${NAME_LINK_GRIPPER_BASE}"
-    name_link_gripper_finger_a="${NAME_LINK_GRIPPER_FINGER_A}"
-    name_link_gripper_finger_b="${NAME_LINK_GRIPPER_FINGER_B}"
-    name_joint_mounting_plate="${NAME_JOINT_MOUNTING_PLATE}"
-    name_joint_base="${NAME_JOINT_BASE}"
-    name_joint_1="${NAME_JOINT_1}"
-    name_joint_2="${NAME_JOINT_2}"
-    name_joint_3="${NAME_JOINT_3}"
-    name_joint_4="${NAME_JOINT_4}"
-    name_joint_5="${NAME_JOINT_5}"
-    name_joint_6="${NAME_JOINT_6}"
-    name_joint_7="${NAME_JOINT_7}"
-    name_joint_cover_2_l="${NAME_JOINT_COVER_2_L}"
-    name_joint_cover_2_r="${NAME_JOINT_COVER_2_R}"
-    name_joint_cover_4_l="${NAME_JOINT_COVER_4_L}"
-    name_joint_cover_4_r="${NAME_JOINT_COVER_4_R}"
-    name_joint_logo_symbol_l="${NAME_JOINT_LOGO_SYMBOL_L}"
-    name_joint_logo_symbol_r="${NAME_JOINT_LOGO_SYMBOL_R}"
-    name_joint_logo_text_l="${NAME_JOINT_LOGO_TEXT_L}"
-    name_joint_logo_text_r="${NAME_JOINT_LOGO_TEXT_R}"
-    name_joint_gripper_finger_a="${NAME_JOINT_GRIPPER_FINGER_A}"
-    name_joint_gripper_finger_b="${NAME_JOINT_GRIPPER_FINGER_B}"
     color_link_base="${COLOR_LINK_BASE}"
     color_link_1="${COLOR_LINK_1}"
@@ -177,12 +99,4 @@
     <xacro:crane_x7_ros2_control_settings
       name="crane_x7"
-      name_joint_1="${NAME_JOINT_1}"
-      name_joint_2="${NAME_JOINT_2}"
-      name_joint_3="${NAME_JOINT_3}"
-      name_joint_4="${NAME_JOINT_4}"
-      name_joint_5="${NAME_JOINT_5}"
-      name_joint_6="${NAME_JOINT_6}"
-      name_joint_7="${NAME_JOINT_7}"
-      name_joint_gripper_finger_a="${NAME_JOINT_GRIPPER_FINGER_A}"
       joint_1_lower_limit="${JOINT_1_LOWER_LIMIT}"
       joint_1_upper_limit="${JOINT_1_UPPER_LIMIT}"
@@ -211,23 +125,4 @@
   <xacro:if value="$(arg use_gazebo)">
     <xacro:gazebo_robot_settings
-      name_link_mounting_plate="${NAME_LINK_MOUNTING_PLATE}"
-      name_link_base="${NAME_LINK_BASE}"
-      name_link_1="${NAME_LINK_1}"
-      name_link_2="${NAME_LINK_2}"
-      name_link_3="${NAME_LINK_3}"
-      name_link_4="${NAME_LINK_4}"
-      name_link_5="${NAME_LINK_5}"
-      name_link_6="${NAME_LINK_6}"
-      name_link_cover_2_l="${NAME_LINK_COVER_2_L}"
-      name_link_cover_2_r="${NAME_LINK_COVER_2_R}"
-      name_link_cover_4_l="${NAME_LINK_COVER_4_L}"
-      name_link_cover_4_r="${NAME_LINK_COVER_4_R}"
-      name_link_logo_symbol_l="${NAME_LINK_LOGO_SYMBOL_L}"
-      name_link_logo_symbol_r="${NAME_LINK_LOGO_SYMBOL_R}"
-      name_link_logo_text_l="${NAME_LINK_LOGO_TEXT_L}"
-      name_link_logo_text_r="${NAME_LINK_LOGO_TEXT_R}"
-      name_link_gripper_base="${NAME_LINK_GRIPPER_BASE}"
-      name_link_gripper_finger_a="${NAME_LINK_GRIPPER_FINGER_A}"
-      name_link_gripper_finger_b="${NAME_LINK_GRIPPER_FINGER_B}"
       config_package="$(arg gz_control_config_package)"
       config_file_path="$(arg gz_control_config_file_path)"
@@ -235,13 +130,4 @@
     <xacro:crane_x7_gazebo_ros2_control_settings
       name="crane_x7"
-      name_joint_1="${NAME_JOINT_1}"
-      name_joint_2="${NAME_JOINT_2}"
-      name_joint_3="${NAME_JOINT_3}"
-      name_joint_4="${NAME_JOINT_4}"
-      name_joint_5="${NAME_JOINT_5}"
-      name_joint_6="${NAME_JOINT_6}"
-      name_joint_7="${NAME_JOINT_7}"
-      name_joint_gripper_finger_a="${NAME_JOINT_GRIPPER_FINGER_A}"
-      name_joint_gripper_finger_b="${NAME_JOINT_GRIPPER_FINGER_B}"
       joint_1_lower_limit="${JOINT_1_LOWER_LIMIT}"
       joint_1_upper_limit="${JOINT_1_UPPER_LIMIT}"

File: urdf/crane_x7.xacro (robot description, xacro)
@@ -25,43 +25,4 @@
   <xacro:macro name="crane_x7"
       params="parent
-              name_link_mounting_plate
-              name_link_base
-              name_link_1
-              name_link_2
-              name_link_3
-              name_link_4
-              name_link_5
-              name_link_6
-              name_link_7
-              name_link_cover_2_l
-              name_link_cover_2_r
-              name_link_cover_4_l
-              name_link_cover_4_r
-              name_link_logo_symbol_l
-              name_link_logo_symbol_r
-              name_link_logo_text_l
-              name_link_logo_text_r
-              name_link_gripper_base
-              name_link_gripper_finger_a
-              name_link_gripper_finger_b
-              name_joint_mounting_plate
-              name_joint_base
-              name_joint_1
-              name_joint_2
-              name_joint_3
-              name_joint_4
-              name_joint_5
-              name_joint_6
-              name_joint_7
-              name_joint_cover_2_l
-              name_joint_cover_2_r
-              name_joint_cover_4_l
-              name_joint_cover_4_r
-              name_joint_logo_symbol_l
-              name_joint_logo_symbol_r
-              name_joint_logo_text_l
-              name_joint_logo_text_r
-              name_joint_gripper_finger_a
-              name_joint_gripper_finger_b
               color_link_base
               color_link_1
@@ -97,6 +58,4 @@
     <xacro:crane_x7_mounting_plate
         parent="${parent}"
-        name_link_mounting_plate="${name_link_mounting_plate}"
-        name_joint_mounting_plate="${name_joint_mounting_plate}"
         color="black">
       <xacro:insert_block name="origin"/>
@@ -104,37 +63,5 @@
     <!-- Arm -->
     <xacro:crane_x7_arm
-        parent="${name_link_mounting_plate}"
-        name_link_base="${name_link_base}"
-        name_link_1="${name_link_1}"
-        name_link_2="${name_link_2}"
-        name_link_3="${name_link_3}"
-        name_link_4="${name_link_4}"
-        name_link_5="${name_link_5}"
-        name_link_6="${name_link_6}"
-        name_link_7="${name_link_7}"
-        name_link_cover_2_l="${name_link_cover_2_l}"
-        name_link_cover_2_r="${name_link_cover_2_r}"
-        name_link_cover_4_l="${name_link_cover_4_l}"
-        name_link_cover_4_r="${name_link_cover_4_r}"
-        name_link_logo_symbol_l="${name_link_logo_symbol_l}"
-        name_link_logo_symbol_r="${name_link_logo_symbol_r}"
-        name_link_logo_text_l="${name_link_logo_text_l}"
-        name_link_logo_text_r="${name_link_logo_text_r}"
-        name_joint_base="${name_joint_base}"
-        name_joint_1="${name_joint_1}"
-        name_joint_2="${name_joint_2}"
-        name_joint_3="${name_joint_3}"
-        name_joint_4="${name_joint_4}"
-        name_joint_5="${name_joint_5}"
-        name_joint_6="${name_joint_6}"
-        name_joint_7="${name_joint_7}"
-        name_joint_cover_2_l="${name_joint_cover_2_l}"
-        name_joint_cover_2_r="${name_joint_cover_2_r}"
-        name_joint_cover_4_l="${name_joint_cover_4_l}"
-        name_joint_cover_4_r="${name_joint_cover_4_r}"
-        name_joint_logo_symbol_l="${name_joint_logo_symbol_l}"
-        name_joint_logo_symbol_r="${name_joint_logo_symbol_r}"
-        name_joint_logo_text_l="${name_joint_logo_text_l}"
-        name_joint_logo_text_r="${name_joint_logo_text_r}"
+      parent="crane_x7_mounting_plate_link"
         color_link_base="${color_link_base}"
         color_link_1="${color_link_1}"
@@ -167,5 +94,5 @@
       <xacro:include filename="$(find realsense2_description)/urdf/_d435.urdf.xacro" />
       <xacro:sensor_d435
-          parent="${name_link_7}"
+          parent="crane_x7_gripper_base_link"
           use_nominal_extrinsics="false"
           add_plug="false"
@@ -176,9 +103,4 @@
     <!-- End effector -->
     <xacro:crane_x7_wide_two_finger_gripper
-        name_link_gripper_base="${name_link_gripper_base}"
-        name_link_gripper_finger_a="${name_link_gripper_finger_a}"
-        name_link_gripper_finger_b="${name_link_gripper_finger_b}"
-        name_joint_gripper_finger_a="${name_joint_gripper_finger_a}"
-        name_joint_gripper_finger_b="${name_joint_gripper_finger_b}"
         color="${color_hand}"
         joint_velocity_limit="${joint_velocity_limit}"
