Commit message: リンクとジョイントのpropertyを廃止

File: urdf/crane_x7_arm.xacro (robot description, xacro)
@@ -6,36 +6,4 @@
   <xacro:macro name="crane_x7_arm"
       params="parent
-              name_link_base
-              name_link_1
-              name_link_2
-              name_link_3
-              name_link_4
-              name_link_5
-              name_link_6
-              name_link_7
-              name_link_cover_2_l
-              name_link_cover_2_r
-              name_link_cover_4_l
-              name_link_cover_4_r
-              name_link_logo_symbol_l
-              name_link_logo_symbol_r
-              name_link_logo_text_l
-              name_link_logo_text_r
-              name_joint_base
-              name_joint_1
-              name_joint_2
-              name_joint_3
-              name_joint_4
-              name_joint_5
-              name_joint_6
-              name_joint_7
-              name_joint_cover_2_l
-              name_joint_cover_2_r
-              name_joint_cover_4_l
-              name_joint_cover_4_r
-              name_joint_logo_symbol_l
-              name_joint_logo_symbol_r
-              name_joint_logo_text_l
-              name_joint_logo_text_r
               color_link_base
               color_link_1
@@ -64,11 +32,11 @@
               *origin">
     <!-- crane_x7_joint_base -->
-    <joint name="${name_joint_base}" type="fixed">
+    <joint name="crane_x7_shoulder_fixed_part_mount_joint" type="fixed">
       <xacro:insert_block name="origin"/>
       <parent link="${parent}"/>
-      <child link="${name_link_base}"/>
+      <child link="crane_x7_shoulder_fixed_part_link"/>
     </joint>
     <!-- crane_x7_link_base -->
-    <link name="${name_link_base}">
+    <link name="crane_x7_shoulder_fixed_part_link">
       <visual>
         <origin xyz="0 0 0" rpy="0 0 0"/>
@@ -95,14 +63,14 @@
     </link>
     <!-- crane_x7_joint_1 -->
-    <joint name="${name_joint_1}" type="revolute">
+    <joint name="crane_x7_shoulder_fixed_part_pan_joint" type="revolute">
       <origin xyz="0 0 0.036" rpy="0 0 0"/>
       <axis xyz="0 0 1"/>
       <limit effort="10.0" velocity="${joint_velocity_limit}" lower="${joint_1_lower_limit}" upper="${joint_1_upper_limit}"/>
-      <parent link="${name_link_base}"/>
-      <child link="${name_link_1}"/>
+      <parent link="crane_x7_shoulder_fixed_part_link"/>
+      <child link="crane_x7_shoulder_revolute_part_link"/>
       <dynamics damping="1.0e-6" friction="2.0e-1"/>
     </joint>
     <!-- crane_x7_link_1 -->
-    <link name="${name_link_1}">
+    <link name="crane_x7_shoulder_revolute_part_link">
       <visual>
         <origin xyz="0 0 0" rpy="0 0 ${M_PI}"/>
@@ -139,14 +107,14 @@
     </link>
     <!-- crane_x7_joint_2 -->
-    <joint name="${name_joint_2}" type="revolute">
+    <joint name="crane_x7_shoulder_revolute_part_tilt_joint" type="revolute">
       <origin xyz="0 0 0.064" rpy="0 0 0"/>
       <axis xyz="0 -1 0"/>
       <limit effort="10.0" velocity="${joint_velocity_limit}" lower="${joint_2_lower_limit}" upper="${joint_2_upper_limit}"/>
-      <parent link="${name_link_1}"/>
-      <child link="${name_link_2}"/>
+      <parent link="crane_x7_shoulder_revolute_part_link"/>
+      <child link="crane_x7_upper_arm_fixed_part_link"/>
       <dynamics damping="1.0e-6" friction="2.0e-1"/>
     </joint>
     <!-- crane_x7_link_2 -->
-    <link name="${name_link_2}">
+    <link name="crane_x7_upper_arm_fixed_part_link">
       <visual>
         <origin xyz="0 0 0" rpy="${M_PI/2} 0 0"/>
@@ -173,11 +141,11 @@
     </link>
     <!-- crane_x7_joint_cover_2_l -->
-    <joint name="${name_joint_cover_2_l}" type="fixed">
-      <parent link="${name_link_2}"/>
-      <child link="${name_link_cover_2_l}"/>
+    <joint name="crane_x7_upper_arm_fixed_part_joint_cover_l_joint" type="fixed">
+      <parent link="crane_x7_upper_arm_fixed_part_link"/>
+      <child link="crane_x7_upper_arm_fixed_part_joint_cover_l_link"/>
       <origin xyz="0 0.0316 0" rpy="0 0 0"/>
     </joint>
     <!-- crane_x7_link_cover_2_l -->
-    <link name="${name_link_cover_2_l}">
+    <link name="crane_x7_upper_arm_fixed_part_joint_cover_l_link">
       <visual>
         <origin xyz="0 0 0" rpy="-${M_PI/2} 0 0"/>
@@ -197,11 +165,11 @@
     </link>
     <!-- crane_x7_joint_cover_2_r -->
-    <joint name="${name_joint_cover_2_r}" type="fixed">
-      <parent link="${name_link_2}"/>
-      <child link="${name_link_cover_2_r}"/>
+    <joint name="crane_x7_upper_arm_fixed_part_joint_cover_r_joint" type="fixed">
+      <parent link="crane_x7_upper_arm_fixed_part_link"/>
+      <child link="crane_x7_upper_arm_fixed_part_joint_cover_r_link"/>
       <origin xyz="0 -0.0316 0" rpy="0 0 0"/>
     </joint>
     <!-- crane_x7_link_cover_2_r -->
-    <link name="${name_link_cover_2_r}">
+    <link name="crane_x7_upper_arm_fixed_part_joint_cover_r_link">
       <visual>
         <origin xyz="0 0 0" rpy="${M_PI/2} 0 0"/>
@@ -221,5 +189,5 @@
     </link>
     <!-- crane_x7_joint_3 -->
-    <joint name="${name_joint_3}" type="revolute">
+    <joint name="crane_x7_upper_arm_revolute_part_twist_joint" type="revolute">
       <origin xyz="0 0 0.065" rpy="0 0 0"/>
       <axis xyz="0 0 1"/>
@@ -228,10 +196,10 @@
           lower="${joint_3_lower_limit}"
           upper="${joint_3_upper_limit}"/>
-      <parent link="${name_link_2}"/>
-      <child link="${name_link_3}"/>
+      <parent link="crane_x7_upper_arm_fixed_part_link"/>
+      <child link="crane_x7_upper_arm_revolute_part_link"/>
       <dynamics damping="1.0e-6" friction="2.0e-1"/>
     </joint>
     <!-- crane_x7_link_3 -->
-    <link name="${name_link_3}">
+    <link name="crane_x7_upper_arm_revolute_part_link">
       <visual>
         <origin xyz="0 0 0" rpy="0 0 0"/>
@@ -258,5 +226,5 @@
     </link>
     <!-- crane_x7_joint_4 -->
-    <joint name="${name_joint_4}" type="revolute">
+    <joint name="crane_x7_upper_arm_revolute_part_rotate_joint" type="revolute">
       <origin xyz="0 0 0.185" rpy="0 0 0"/>
       <axis xyz="0 -1 0"/>
@@ -265,10 +233,10 @@
           lower="${joint_4_lower_limit}"
           upper="${joint_4_upper_limit}"/>
-      <parent link="${name_link_3}"/>
-      <child link="${name_link_4}"/>
+      <parent link="crane_x7_upper_arm_revolute_part_link"/>
+      <child link="crane_x7_lower_arm_fixed_part_link"/>
       <dynamics damping="1.0e-6" friction="2.0e-1"/>
     </joint>
     <!-- crane_x7_link_4 -->
-    <link name="${name_link_4}">
+    <link name="crane_x7_lower_arm_fixed_part_link">
       <visual>
         <origin xyz="0 0 0" rpy="${M_PI/2} 0 0"/>
@@ -295,11 +263,11 @@
     </link>
     <!-- crane_x7_joint_cover_4_l -->
-    <joint name="${name_joint_cover_4_l}" type="fixed">
-      <parent link="${name_link_4}"/>
-      <child link="${name_link_cover_4_l}"/>
+    <joint name="crane_x7_lower_arm_fixed_part_joint_cover_l_joint" type="fixed">
+      <parent link="crane_x7_lower_arm_fixed_part_link"/>
+      <child link="crane_x7_lower_arm_fixed_part_joint_cover_l_link"/>
       <origin xyz="0 0.025 0" rpy="0 0 0"/>
     </joint>
     <!-- crane_x7_link_cover_4_l -->
-    <link name="${name_link_cover_4_l}">
+    <link name="crane_x7_lower_arm_fixed_part_joint_cover_l_link">
       <visual>
         <origin xyz="0 0 0" rpy="-${M_PI/2} 0 0"/>
@@ -319,11 +287,11 @@
     </link>
     <!-- crane_x7_joint_cover_4_r -->
-    <joint name="${name_joint_cover_4_r}" type="fixed">
-      <parent link="${name_link_4}"/>
-      <child link="${name_link_cover_4_r}"/>
+    <joint name="crane_x7_lower_arm_fixed_part_joint_cover_r_joint" type="fixed">
+      <parent link="crane_x7_lower_arm_fixed_part_link"/>
+      <child link="crane_x7_lower_arm_fixed_part_joint_cover_r_link"/>
       <origin xyz="0 -0.025 0" rpy="0 0 0"/>
     </joint>
     <!-- crane_x7_link_cover_4_r -->
-    <link name="${name_link_cover_4_r}">
+    <link name="crane_x7_lower_arm_fixed_part_joint_cover_r_link">
       <visual>
         <origin xyz="0 0 0" rpy="${M_PI/2} 0 0"/>
@@ -343,14 +311,14 @@
     </link>
     <!-- crane_x7_joint_5 -->
-    <joint name="${name_joint_5}" type="revolute">
+    <joint name="crane_x7_lower_arm_fixed_part_joint" type="revolute">
       <origin xyz="0 0 0.121" rpy="0 0 0"/>
       <axis xyz="0 0 1"/>
       <limit effort="4.0" velocity="${joint_velocity_limit}" lower="${joint_5_lower_limit}" upper="${joint_5_upper_limit}"/>
-      <parent link="${name_link_4}"/>
-      <child link="${name_link_5}"/>
+      <parent link="crane_x7_lower_arm_fixed_part_link"/>
+      <child link="crane_x7_lower_arm_revolute_part_link"/>
       <dynamics damping="1.0e-6" friction="2.0e-1"/>
     </joint>
     <!-- crane_x7_link_5 -->
-    <link name="${name_link_5}">
+    <link name="crane_x7_lower_arm_revolute_part_link">
       <visual>
         <origin xyz="0 0 0" rpy="0 0 0"/>
@@ -378,24 +346,16 @@
     <!-- logo -->
     <xacro:crane_x7_logos
-      parent="${name_link_5}"
-      name_link_logo_symbol_l="${name_link_logo_symbol_l}"
-      name_link_logo_symbol_r="${name_link_logo_symbol_r}"
-      name_link_logo_text_l="${name_link_logo_text_l}"
-      name_link_logo_text_r="${name_link_logo_text_r}"
-      name_joint_logo_symbol_l="${name_joint_logo_symbol_l}"
-      name_joint_logo_symbol_r="${name_joint_logo_symbol_r}"
-      name_joint_logo_text_l="${name_joint_logo_text_l}"
-      name_joint_logo_text_r="${name_joint_logo_text_r}"/>
+      parent="crane_x7_lower_arm_revolute_part_link"/>
     <!-- crane_x7_joint_6 -->
-    <joint name="${name_joint_6}" type="revolute">
+    <joint name="crane_x7_lower_arm_revolute_part_joint" type="revolute">
       <origin xyz="0 0 0.129" rpy="0 0 0"/>
       <axis xyz="0 -1 0"/>
       <limit effort="4.0" velocity="${joint_velocity_limit}" lower="${joint_6_lower_limit}" upper="${joint_6_upper_limit}"/>
-      <parent link="${name_link_5}"/>
-      <child link="${name_link_6}"/>
+      <parent link="crane_x7_lower_arm_revolute_part_link"/>
+      <child link="crane_x7_wrist_link"/>
       <dynamics damping="1.0e-6" friction="2.0e-1"/>
     </joint>
     <!-- crane_x7_link_6 -->
-    <link name="${name_link_6}">
+    <link name="crane_x7_wrist_link">
       <visual>
         <origin xyz="0 0 0" rpy="${M_PI/2} 0 0"/>
@@ -422,10 +382,10 @@
     </link>
     <!-- crane_x7_joint_7 -->
-    <joint name="${name_joint_7}" type="revolute">
+    <joint name="crane_x7_wrist_joint" type="revolute">
       <origin xyz="0 0 0.019" rpy="0 0 0"/>
       <axis xyz="0 0 1"/>
       <limit effort="4.0" velocity="${joint_velocity_limit}" lower="${joint_7_lower_limit}" upper="${joint_7_upper_limit}"/>
-      <parent link="${name_link_6}"/>
-      <child link="${name_link_7}"/>
+      <parent link="crane_x7_wrist_link"/>
+      <child link="crane_x7_gripper_base_link"/>
       <dynamics damping="1.0e-6" friction="2.0e-1"/>
     </joint>

File: urdf/crane_x7_mounting_plate.xacro (robot description, xacro)
@@ -7,14 +7,12 @@
   <xacro:macro name="crane_x7_mounting_plate"
       params="parent
-              name_link_mounting_plate
-              name_joint_mounting_plate
               color
               *origin">
-    <joint name="${name_joint_mounting_plate}" type="fixed">
+    <joint name="crane_x7_mounting_plate_joint" type="fixed">
       <xacro:insert_block name="origin"/>
       <parent link="${parent}"/>
-      <child link="${name_link_mounting_plate}"/>
+      <child link="crane_x7_mounting_plate_link"/>
     </joint>
-    <link name="${name_link_mounting_plate}">
+    <link name="crane_x7_mounting_plate_link">
       <visual>
         <origin xyz="0 0 0" rpy="0 0 0"/>

File: urdf/crane_x7_rt_logos.xacro (robot description, xacro)
@@ -2,15 +2,7 @@
 <robot xmlns:xacro="http://ros.org/wiki/xacro">
   <xacro:macro name="crane_x7_logos"
-      params="parent
-              name_link_logo_symbol_l
-              name_link_logo_symbol_r
-              name_link_logo_text_l
-              name_link_logo_text_r
-              name_joint_logo_symbol_l
-              name_joint_logo_symbol_r
-              name_joint_logo_text_l
-              name_joint_logo_text_r">
+      params="parent">
     <!-- Left side logo text -->
-    <link name="${name_link_logo_text_l}">
+    <link name="crane_x7_lower_arm_revolute_part_logo_text_l_link">
       <visual>
         <origin xyz="0 0 0" rpy="-${M_PI/2} ${M_PI/2} 0"/>
@@ -29,11 +21,11 @@
       </collision>
     </link>
-    <joint name="${name_joint_logo_text_l}" type="fixed">
+    <joint name="crane_x7_lower_arm_revolute_part_logo_text_l_joint" type="fixed">
       <parent link="${parent}"/>
-      <child link="${name_link_logo_text_l}"/>
+      <child link="crane_x7_lower_arm_revolute_part_logo_text_l_link"/>
       <origin xyz="0 0.0345 0.095" rpy="0 0 0"/>
     </joint>
     <!-- Left side logo symbol -->
-    <link name="${name_link_logo_symbol_l}">
+    <link name="crane_x7_lower_arm_revolute_part_logo_symbol_l_link">
       <visual>
         <origin xyz="0 0 0" rpy="-${M_PI/2} ${M_PI/2} 0"/>
@@ -52,11 +44,11 @@
       </collision>
     </link>
-    <joint name="${name_joint_logo_symbol_l}" type="fixed">
+    <joint name="crane_x7_lower_arm_revolute_part_logo_symbol_l_joint" type="fixed">
       <parent link="${parent}"/>
-      <child link="${name_link_logo_symbol_l}"/>
+      <child link="crane_x7_lower_arm_revolute_part_logo_symbol_l_link"/>
       <origin xyz="0 0.0345 0.132" rpy="0 0 0"/>
     </joint>
     <!-- Right side logo text -->
-    <link name="${name_link_logo_text_r}">
+    <link name="crane_x7_lower_arm_revolute_part_logo_text_r_link">
       <visual>
         <origin xyz="0 0 0" rpy="${M_PI/2} -${M_PI/2} 0"/>
@@ -75,11 +67,11 @@
       </collision>
     </link>
-    <joint name="${name_joint_logo_text_r}" type="fixed">
+    <joint name="crane_x7_lower_arm_revolute_part_logo_text_r_joint" type="fixed">
       <parent link="${parent}"/>
-      <child link="${name_link_logo_text_r}"/>
+      <child link="crane_x7_lower_arm_revolute_part_logo_text_r_link"/>
       <origin xyz="0 -0.0345 0.104" rpy="0 0 0"/>
     </joint>
     <!-- Right side logo symbol -->
-    <link name="${name_link_logo_symbol_r}">
+    <link name="crane_x7_lower_arm_revolute_part_logo_symbol_r_link">
       <visual>
         <origin xyz="0 0 0" rpy="${M_PI/2} -${M_PI/2} 0"/>
@@ -98,7 +90,7 @@
       </collision>
     </link>
-    <joint name="${name_joint_logo_symbol_r}" type="fixed">
+    <joint name="crane_x7_lower_arm_revolute_part_logo_symbol_r_joint" type="fixed">
       <parent link="${parent}"/>
-      <child link="${name_link_logo_symbol_r}"/>
+      <child link="crane_x7_lower_arm_revolute_part_logo_symbol_r_link"/>
       <origin xyz="0 -0.0345 0.065" rpy="0 0 0"/>
     </joint>

File: urdf/crane_x7_wide_two_finger_gripper.xacro (robot description, xacro)
@@ -5,14 +5,9 @@
   <xacro:property name="SCALE_CM" value="0.01"/>
   <xacro:macro name="crane_x7_wide_two_finger_gripper"
-    params="name_link_gripper_base
-            name_link_gripper_finger_a
-            name_link_gripper_finger_b
-            name_joint_gripper_finger_a
-            name_joint_gripper_finger_b
-            color
+    params="color
             joint_velocity_limit
             joint_hand_lower_limit
             joint_hand_upper_limit">
-    <link name="${name_link_gripper_base}">
+    <link name="crane_x7_gripper_base_link">
       <visual>
         <origin xyz="0 0 0" rpy="0 0 0"/>
@@ -38,13 +33,13 @@
       </inertial>
     </link>
-    <joint name="${name_joint_gripper_finger_a}" type="revolute">
+    <joint name="crane_x7_gripper_finger_a_joint" type="revolute">
       <origin xyz="-0.012 0.0 0.024" rpy="0 0 0"/>
       <axis xyz="0 -1 0"/>
       <limit effort="4.0" velocity="${joint_velocity_limit}" lower="${joint_hand_lower_limit}" upper="${joint_hand_upper_limit}"/>
-      <parent link="${name_link_gripper_base}"/>
-      <child link="${name_link_gripper_finger_a}"/>
+      <parent link="crane_x7_gripper_base_link"/>
+      <child link="crane_x7_gripper_finger_a_link"/>
       <dynamics damping="1.0e-6" friction="8.0e-1"/>
     </joint>
-    <link name="${name_link_gripper_finger_a}">
+    <link name="crane_x7_gripper_finger_a_link">
       <visual>
         <origin xyz="0 0 0" rpy="${M_PI/2} 0 0"/>
@@ -70,14 +65,14 @@
       </inertial>
     </link>
-    <joint name="${name_joint_gripper_finger_b}" type="revolute">
+    <joint name="crane_x7_gripper_finger_b_joint" type="revolute">
       <origin xyz="0.012 0.0 0.024" rpy="0 0 0"/>
       <axis xyz="0 1 0"/>
       <limit effort="4.0" velocity="${joint_velocity_limit}" lower="${joint_hand_lower_limit}" upper="${joint_hand_upper_limit}"/>
-      <parent link="${name_link_gripper_base}"/>
-      <child link="${name_link_gripper_finger_b}"/>
-      <mimic joint="${name_joint_gripper_finger_a}"/>
+      <parent link="crane_x7_gripper_base_link"/>
+      <child link="crane_x7_gripper_finger_b_link"/>
+      <mimic joint="crane_x7_gripper_finger_a_joint"/>
       <dynamics damping="1.0e-6" friction="8.0e-1"/>
     </joint>
-    <link name="${name_link_gripper_finger_b}">
+    <link name="crane_x7_gripper_finger_b_link">
       <visual>
         <origin xyz="0 0 0" rpy="${M_PI/2} 0 0"/>
