Commit message: 不要な変数を削除

File: urdf/crane_x7_arm.xacro (robot description, xacro)
@@ -1,6 +1,4 @@
 <?xml version="1.0"?>
 <robot xmlns:xacro="http://ros.org/wiki/xacro">
-  <xacro:property name="SCALE_MM" value="0.001"/>
-  <xacro:property name="SCALE_CM" value="0.01"/>
   <!-- Macro for the standard CRANE-X7 configuration -->
   <xacro:macro name="crane_x7_arm" params="parent *origin">

File: urdf/crane_x7_mounting_plate.xacro (robot description, xacro)
@@ -1,7 +1,4 @@
 <?xml version="1.0"?>
 <robot xmlns:xacro="http://ros.org/wiki/xacro">
-  <xacro:property name="M_PI" value="3.14159"/>
-  <xacro:property name="SCALE_MM" value="0.001"/>
-  <xacro:property name="SCALE_CM" value="0.01"/>
   <xacro:property name="MOUNTING_PLATE_THICKNESS" value="0.005"/>
   <xacro:macro name="crane_x7_mounting_plate" params="parent color *origin">

File: urdf/crane_x7_wide_two_finger_gripper.xacro (robot description, xacro)
@@ -1,7 +1,4 @@
 <?xml version="1.0"?>
 <robot xmlns:xacro="http://ros.org/wiki/xacro">
-  <xacro:property name="M_PI" value="3.14159"/>
-  <xacro:property name="SCALE_MM" value="0.001"/>
-  <xacro:property name="SCALE_CM" value="0.01"/>
   <xacro:macro name="crane_x7_wide_two_finger_gripper">
     <link name="${NAME_LINK_GRIPPER_BASE}">
