Commit message: crane_x7マクロとそこで呼び出されるマクロのパラメータを削除

File: urdf/crane_x7.urdf.xacro (robot description, xacro)
@@ -16,4 +16,13 @@
   <xacro:arg name="gz_control_config_package" default="" />
   <xacro:arg name="gz_control_config_file_path" default="" />
+  <xacro:property name="USE_D435" value="$(arg use_d435)"/>
+  <xacro:property name="USE_MOCK_COMPONENTS" value="$(arg use_mock_components)"/>
+  <xacro:property name="PORT_NAME" value="$(arg port_name)"/>
+  <xacro:property name="BAUDRATE" value="$(arg baudrate)"/>
+  <xacro:property name="TIMEOUT_SECONDS" value="$(arg timeout_seconds)"/>
+  <xacro:property name="MANIPULATOR_CONFIG_FILE_PATH" value="$(arg manipulator_config_file_path)"/>
+  <xacro:property name="MANIPULATOR_LINKS_FILE_PATH" value="$(arg manipulator_links_file_path)"/>
+  <xacro:property name="GZ_CONTROL_CONFIG_PACKAGE" value="$(arg gz_control_config_package)"/>
+  <xacro:property name="GZ_CONTROL_CONFIG_FILE_PATH" value="$(arg gz_control_config_file_path)"/>
   <xacro:property name="M_PI" value="3.14159"/>
   <xacro:property name="NAME_LINK_MOUNTING_PLATE" value="crane_x7_mounting_plate_link"/>
@@ -97,74 +106,6 @@
        allows accessing different operational areas, e.g. left-handed vs.
        right-handed robots. -->
-  <xacro:crane_x7
-    parent="base_link"
-    name_link_mounting_plate="${NAME_LINK_MOUNTING_PLATE}"
-    name_link_base="${NAME_LINK_BASE}"
-    name_link_1="${NAME_LINK_1}"
-    name_link_2="${NAME_LINK_2}"
-    name_link_3="${NAME_LINK_3}"
-    name_link_4="${NAME_LINK_4}"
-    name_link_5="${NAME_LINK_5}"
-    name_link_6="${NAME_LINK_6}"
-    name_link_7="${NAME_LINK_7}"
-    name_link_cover_2_l="${NAME_LINK_COVER_2_L}"
-    name_link_cover_2_r="${NAME_LINK_COVER_2_R}"
-    name_link_cover_4_l="${NAME_LINK_COVER_4_L}"
-    name_link_cover_4_r="${NAME_LINK_COVER_4_R}"
-    name_link_logo_symbol_l="${NAME_LINK_LOGO_SYMBOL_L}"
-    name_link_logo_symbol_r="${NAME_LINK_LOGO_SYMBOL_R}"
-    name_link_logo_text_l="${NAME_LINK_LOGO_TEXT_L}"
-    name_link_logo_text_r="${NAME_LINK_LOGO_TEXT_R}"
-    name_link_gripper_base="${NAME_LINK_GRIPPER_BASE}"
-    name_link_gripper_finger_a="${NAME_LINK_GRIPPER_FINGER_A}"
-    name_link_gripper_finger_b="${NAME_LINK_GRIPPER_FINGER_B}"
-    name_joint_mounting_plate="${NAME_JOINT_MOUNTING_PLATE}"
-    name_joint_base="${NAME_JOINT_BASE}"
-    name_joint_1="${NAME_JOINT_1}"
-    name_joint_2="${NAME_JOINT_2}"
-    name_joint_3="${NAME_JOINT_3}"
-    name_joint_4="${NAME_JOINT_4}"
-    name_joint_5="${NAME_JOINT_5}"
-    name_joint_6="${NAME_JOINT_6}"
-    name_joint_7="${NAME_JOINT_7}"
-    name_joint_cover_2_l="${NAME_JOINT_COVER_2_L}"
-    name_joint_cover_2_r="${NAME_JOINT_COVER_2_R}"
-    name_joint_cover_4_l="${NAME_JOINT_COVER_4_L}"
-    name_joint_cover_4_r="${NAME_JOINT_COVER_4_R}"
-    name_joint_logo_symbol_l="${NAME_JOINT_LOGO_SYMBOL_L}"
-    name_joint_logo_symbol_r="${NAME_JOINT_LOGO_SYMBOL_R}"
-    name_joint_logo_text_l="${NAME_JOINT_LOGO_TEXT_L}"
-    name_joint_logo_text_r="${NAME_JOINT_LOGO_TEXT_R}"
-    name_joint_gripper_finger_a="${NAME_JOINT_GRIPPER_FINGER_A}"
-    name_joint_gripper_finger_b="${NAME_JOINT_GRIPPER_FINGER_B}"
-    color_link_base="${COLOR_LINK_BASE}"
-    color_link_1="${COLOR_LINK_1}"
-    color_link_cover_2="${COLOR_LINK_COVER_2}"
-    color_link_2="${COLOR_LINK_2}"
-    color_link_3="${COLOR_LINK_3}"
-    color_link_cover_4="${COLOR_LINK_COVER_4}"
-    color_link_4="${COLOR_LINK_4}"
-    color_link_5="${COLOR_LINK_5}"
-    color_link_6="${COLOR_LINK_6}"
-    color_hand="${COLOR_HAND}"
-    joint_velocity_limit="${JOINT_VELOCITY_LIMIT}"
-    joint_1_lower_limit="${JOINT_1_LOWER_LIMIT}"
-    joint_1_upper_limit="${JOINT_1_UPPER_LIMIT}"
-    joint_2_lower_limit="${JOINT_2_LOWER_LIMIT}"
-    joint_2_upper_limit="${JOINT_2_UPPER_LIMIT}"
-    joint_3_lower_limit="${JOINT_3_LOWER_LIMIT}"
-    joint_3_upper_limit="${JOINT_3_UPPER_LIMIT}"
-    joint_4_lower_limit="${JOINT_4_LOWER_LIMIT}"
-    joint_4_upper_limit="${JOINT_4_UPPER_LIMIT}"
-    joint_5_lower_limit="${JOINT_5_LOWER_LIMIT}"
-    joint_5_upper_limit="${JOINT_5_UPPER_LIMIT}"
-    joint_6_lower_limit="${JOINT_6_LOWER_LIMIT}"
-    joint_6_upper_limit="${JOINT_6_UPPER_LIMIT}"
-    joint_7_lower_limit="${JOINT_7_LOWER_LIMIT}"
-    joint_7_upper_limit="${JOINT_7_UPPER_LIMIT}"
-    joint_hand_lower_limit="${JOINT_HAND_LOWER_LIMIT}"
-    joint_hand_upper_limit="${JOINT_HAND_UPPER_LIMIT}"
-    use_d435="$(arg use_d435)">
-    <origin xyz="0 0 0"/>
+  <xacro:crane_x7 parent="base_link">
+    <origin xyz="0 0 0" rpy="0 0 0"/>
   </xacro:crane_x7>
   <xacro:unless value="$(arg use_gazebo)">

File: urdf/crane_x7.xacro (robot description, xacro)
@@ -23,149 +23,19 @@
     <color rgba="0.3 0.3 1.0 1.0"/>
   </material>
-  <xacro:macro name="crane_x7"
-      params="parent
-              name_link_mounting_plate
-              name_link_base
-              name_link_1
-              name_link_2
-              name_link_3
-              name_link_4
-              name_link_5
-              name_link_6
-              name_link_7
-              name_link_cover_2_l
-              name_link_cover_2_r
-              name_link_cover_4_l
-              name_link_cover_4_r
-              name_link_logo_symbol_l
-              name_link_logo_symbol_r
-              name_link_logo_text_l
-              name_link_logo_text_r
-              name_link_gripper_base
-              name_link_gripper_finger_a
-              name_link_gripper_finger_b
-              name_joint_mounting_plate
-              name_joint_base
-              name_joint_1
-              name_joint_2
-              name_joint_3
-              name_joint_4
-              name_joint_5
-              name_joint_6
-              name_joint_7
-              name_joint_cover_2_l
-              name_joint_cover_2_r
-              name_joint_cover_4_l
-              name_joint_cover_4_r
-              name_joint_logo_symbol_l
-              name_joint_logo_symbol_r
-              name_joint_logo_text_l
-              name_joint_logo_text_r
-              name_joint_gripper_finger_a
-              name_joint_gripper_finger_b
-              color_link_base
-              color_link_1
-              color_link_cover_2
-              color_link_2
-              color_link_3
-              color_link_cover_4
-              color_link_4
-              color_link_5
-              color_link_6
-              color_hand
-              joint_velocity_limit
-              joint_1_lower_limit
-              joint_1_upper_limit
-              joint_2_lower_limit
-              joint_2_upper_limit
-              joint_3_lower_limit
-              joint_3_upper_limit
-              joint_4_lower_limit
-              joint_4_upper_limit
-              joint_5_lower_limit
-              joint_5_upper_limit
-              joint_6_lower_limit
-              joint_6_upper_limit
-              joint_7_lower_limit
-              joint_7_upper_limit
-              joint_hand_lower_limit
-              joint_hand_upper_limit
-              use_d435
-              *origin">
+  <xacro:macro name="crane_x7" params="parent *origin">
     <!-- Mounting plate
          (Root of the manipulator's TF tree) -->
-    <xacro:crane_x7_mounting_plate
-        parent="${parent}"
-        name_link_mounting_plate="${name_link_mounting_plate}"
-        name_joint_mounting_plate="${name_joint_mounting_plate}"
-        color="black">
+    <xacro:crane_x7_mounting_plate parent="${parent}" color="black">
       <xacro:insert_block name="origin"/>
     </xacro:crane_x7_mounting_plate>
     <!-- Arm -->
-    <xacro:crane_x7_arm
-        parent="${name_link_mounting_plate}"
-        name_link_base="${name_link_base}"
-        name_link_1="${name_link_1}"
-        name_link_2="${name_link_2}"
-        name_link_3="${name_link_3}"
-        name_link_4="${name_link_4}"
-        name_link_5="${name_link_5}"
-        name_link_6="${name_link_6}"
-        name_link_7="${name_link_7}"
-        name_link_cover_2_l="${name_link_cover_2_l}"
-        name_link_cover_2_r="${name_link_cover_2_r}"
-        name_link_cover_4_l="${name_link_cover_4_l}"
-        name_link_cover_4_r="${name_link_cover_4_r}"
-        name_link_logo_symbol_l="${name_link_logo_symbol_l}"
-        name_link_logo_symbol_r="${name_link_logo_symbol_r}"
-        name_link_logo_text_l="${name_link_logo_text_l}"
-        name_link_logo_text_r="${name_link_logo_text_r}"
-        name_joint_base="${name_joint_base}"
-        name_joint_1="${name_joint_1}"
-        name_joint_2="${name_joint_2}"
-        name_joint_3="${name_joint_3}"
-        name_joint_4="${name_joint_4}"
-        name_joint_5="${name_joint_5}"
-        name_joint_6="${name_joint_6}"
-        name_joint_7="${name_joint_7}"
-        name_joint_cover_2_l="${name_joint_cover_2_l}"
-        name_joint_cover_2_r="${name_joint_cover_2_r}"
-        name_joint_cover_4_l="${name_joint_cover_4_l}"
-        name_joint_cover_4_r="${name_joint_cover_4_r}"
-        name_joint_logo_symbol_l="${name_joint_logo_symbol_l}"
-        name_joint_logo_symbol_r="${name_joint_logo_symbol_r}"
-        name_joint_logo_text_l="${name_joint_logo_text_l}"
-        name_joint_logo_text_r="${name_joint_logo_text_r}"
-        color_link_base="${color_link_base}"
-        color_link_1="${color_link_1}"
-        color_link_cover_2="${color_link_cover_2}"
-        color_link_2="${color_link_2}"
-        color_link_3="${color_link_3}"
-        color_link_cover_4="${color_link_cover_4}"
-        color_link_4="${color_link_4}"
-        color_link_5="${color_link_5}"
-        color_link_6="${color_link_6}"
-        joint_velocity_limit="${joint_velocity_limit}"
-        joint_1_lower_limit="${joint_1_lower_limit}"
-        joint_1_upper_limit="${joint_1_upper_limit}"
-        joint_2_lower_limit="${joint_2_lower_limit}"
-        joint_2_upper_limit="${joint_2_upper_limit}"
-        joint_3_lower_limit="${joint_3_lower_limit}"
-        joint_3_upper_limit="${joint_3_upper_limit}"
-        joint_4_lower_limit="${joint_4_lower_limit}"
-        joint_4_upper_limit="${joint_4_upper_limit}"
-        joint_5_lower_limit="${joint_5_lower_limit}"
-        joint_5_upper_limit="${joint_5_upper_limit}"
-        joint_6_lower_limit="${joint_6_lower_limit}"
-        joint_6_upper_limit="${joint_6_upper_limit}"
-        joint_7_lower_limit="${joint_7_lower_limit}"
-        joint_7_upper_limit="${joint_7_upper_limit}">
+    <xacro:crane_x7_arm parent="${NAME_LINK_MOUNTING_PLATE}">
       <origin xyz="0 0 ${MOUNTING_PLATE_THICKNESS}" rpy="0 0 0"/>
     </xacro:crane_x7_arm>
     <!-- RealSense D435 -->
-    <xacro:if value="$(arg use_d435)">
+    <xacro:if value="${USE_D435}">
       <xacro:include filename="$(find realsense2_description)/urdf/_d435.urdf.xacro" />
       <xacro:sensor_d435
-          parent="${name_link_7}"
+          parent="${NAME_LINK_7}"
           use_nominal_extrinsics="false"
           add_plug="false"
@@ -175,14 +45,5 @@
     </xacro:if>
     <!-- End effector -->
-    <xacro:crane_x7_wide_two_finger_gripper
-        name_link_gripper_base="${name_link_gripper_base}"
-        name_link_gripper_finger_a="${name_link_gripper_finger_a}"
-        name_link_gripper_finger_b="${name_link_gripper_finger_b}"
-        name_joint_gripper_finger_a="${name_joint_gripper_finger_a}"
-        name_joint_gripper_finger_b="${name_joint_gripper_finger_b}"
-        color="${color_hand}"
-        joint_velocity_limit="${joint_velocity_limit}"
-        joint_hand_lower_limit="${joint_hand_lower_limit}"
-        joint_hand_upper_limit="${joint_hand_upper_limit}"/>
+    <xacro:crane_x7_wide_two_finger_gripper/>
   </xacro:macro>
 </robot>
