Commit message: crane_x7マクロとそこで呼び出されるマクロのパラメータを削除

File: urdf/crane_x7_arm.xacro (robot description, xacro)
@@ -4,71 +4,13 @@
   <xacro:property name="SCALE_CM" value="0.01"/>
   <!-- Macro for the standard CRANE-X7 configuration -->
-  <xacro:macro name="crane_x7_arm"
-      params="parent
-              name_link_base
-              name_link_1
-              name_link_2
-              name_link_3
-              name_link_4
-              name_link_5
-              name_link_6
-              name_link_7
-              name_link_cover_2_l
-              name_link_cover_2_r
-              name_link_cover_4_l
-              name_link_cover_4_r
-              name_link_logo_symbol_l
-              name_link_logo_symbol_r
-              name_link_logo_text_l
-              name_link_logo_text_r
-              name_joint_base
-              name_joint_1
-              name_joint_2
-              name_joint_3
-              name_joint_4
-              name_joint_5
-              name_joint_6
-              name_joint_7
-              name_joint_cover_2_l
-              name_joint_cover_2_r
-              name_joint_cover_4_l
-              name_joint_cover_4_r
-              name_joint_logo_symbol_l
-              name_joint_logo_symbol_r
-              name_joint_logo_text_l
-              name_joint_logo_text_r
-              color_link_base
-              color_link_1
-              color_link_cover_2
-              color_link_2
-              color_link_3
-              color_link_cover_4
-              color_link_4
-              color_link_5
-              color_link_6
-              joint_velocity_limit
-              joint_1_lower_limit
-              joint_1_upper_limit
-              joint_2_lower_limit
-              joint_2_upper_limit
-              joint_3_lower_limit
-              joint_3_upper_limit
-              joint_4_lower_limit
-              joint_4_upper_limit
-              joint_5_lower_limit
-              joint_5_upper_limit
-              joint_6_lower_limit
-              joint_6_upper_limit
-              joint_7_lower_limit
-              joint_7_upper_limit
-              *origin">
+  <xacro:macro name="crane_x7_arm" params="parent *origin">
     <!-- crane_x7_joint_base -->
-    <joint name="${name_joint_base}" type="fixed">
+    <joint name="${NAME_JOINT_BASE}" type="fixed">
       <xacro:insert_block name="origin"/>
       <parent link="${parent}"/>
-      <child link="${name_link_base}"/>
+      <child link="${NAME_LINK_BASE}"/>
     </joint>
     <!-- crane_x7_link_base -->
-    <link name="${name_link_base}">
+    <link name="${NAME_LINK_BASE}">
       <visual>
         <origin xyz="0 0 0" rpy="0 0 0"/>
@@ -77,5 +19,5 @@
               scale="1 1 1"/>
         </geometry>
-        <material name="${color_link_base}"/>
+        <material name="${COLOR_LINK_BASE}"/>
       </visual>
       <collision>
@@ -95,14 +37,19 @@
     </link>
     <!-- crane_x7_joint_1 -->
-    <joint name="${name_joint_1}" type="revolute">
+    <joint name="${NAME_JOINT_1}" type="revolute">
       <origin xyz="0 0 0.036" rpy="0 0 0"/>
       <axis xyz="0 0 1"/>
-      <limit effort="10.0" velocity="${joint_velocity_limit}" lower="${joint_1_lower_limit}" upper="${joint_1_upper_limit}"/>
-      <parent link="${name_link_base}"/>
-      <child link="${name_link_1}"/>
+      <limit
+        effort="10.0"
+        velocity="${JOINT_VELOCITY_LIMIT}"
+        lower="${JOINT_1_LOWER_LIMIT}"
+        upper="${JOINT_1_UPPER_LIMIT}"
+        />
+      <parent link="${NAME_LINK_BASE}"/>
+      <child link="${NAME_LINK_1}"/>
       <dynamics damping="1.0e-6" friction="2.0e-1"/>
     </joint>
     <!-- crane_x7_link_1 -->
-    <link name="${name_link_1}">
+    <link name="${NAME_LINK_1}">
       <visual>
         <origin xyz="0 0 0" rpy="0 0 ${M_PI}"/>
@@ -111,5 +58,5 @@
               scale="1 1 1"/>
         </geometry>
-        <material name="${color_link_1}"/>
+        <material name="${COLOR_LINK_1}"/>
       </visual>
       <collision>
@@ -139,14 +86,19 @@
     </link>
     <!-- crane_x7_joint_2 -->
-    <joint name="${name_joint_2}" type="revolute">
+    <joint name="${NAME_JOINT_2}" type="revolute">
       <origin xyz="0 0 0.064" rpy="0 0 0"/>
       <axis xyz="0 -1 0"/>
-      <limit effort="10.0" velocity="${joint_velocity_limit}" lower="${joint_2_lower_limit}" upper="${joint_2_upper_limit}"/>
-      <parent link="${name_link_1}"/>
-      <child link="${name_link_2}"/>
+      <limit
+        effort="10.0"
+        velocity="${JOINT_VELOCITY_LIMIT}"
+        lower="${JOINT_2_LOWER_LIMIT}"
+        upper="${JOINT_2_UPPER_LIMIT}"
+        />
+      <parent link="${NAME_LINK_1}"/>
+      <child link="${NAME_LINK_2}"/>
       <dynamics damping="1.0e-6" friction="2.0e-1"/>
     </joint>
     <!-- crane_x7_link_2 -->
-    <link name="${name_link_2}">
+    <link name="${NAME_LINK_2}">
       <visual>
         <origin xyz="0 0 0" rpy="${M_PI/2} 0 0"/>
@@ -155,5 +107,5 @@
               scale="1 1 1"/>
         </geometry>
-        <material name="${color_link_2}"/>
+        <material name="${COLOR_LINK_2}"/>
       </visual>
       <collision>
@@ -173,11 +125,11 @@
     </link>
     <!-- crane_x7_joint_cover_2_l -->
-    <joint name="${name_joint_cover_2_l}" type="fixed">
-      <parent link="${name_link_2}"/>
-      <child link="${name_link_cover_2_l}"/>
+    <joint name="${NAME_JOINT_COVER_2_L}" type="fixed">
+      <parent link="${NAME_LINK_2}"/>
+      <child link="${NAME_LINK_COVER_2_L}"/>
       <origin xyz="0 0.0316 0" rpy="0 0 0"/>
     </joint>
     <!-- crane_x7_link_cover_2_l -->
-    <link name="${name_link_cover_2_l}">
+    <link name="${NAME_LINK_COVER_2_L}">
       <visual>
         <origin xyz="0 0 0" rpy="-${M_PI/2} 0 0"/>
@@ -186,5 +138,5 @@
               scale="1 1 1"/>
         </geometry>
-        <material name="${color_link_cover_2}"/>
+        <material name="${COLOR_LINK_COVER_2}"/>
       </visual>
       <collision>
@@ -197,18 +149,18 @@
     </link>
     <!-- crane_x7_joint_cover_2_r -->
-    <joint name="${name_joint_cover_2_r}" type="fixed">
-      <parent link="${name_link_2}"/>
-      <child link="${name_link_cover_2_r}"/>
+    <joint name="${NAME_JOINT_COVER_2_R}" type="fixed">
+      <parent link="${NAME_LINK_2}"/>
+      <child link="${NAME_LINK_COVER_2_R}"/>
       <origin xyz="0 -0.0316 0" rpy="0 0 0"/>
     </joint>
     <!-- crane_x7_link_cover_2_r -->
-    <link name="${name_link_cover_2_r}">
-      <visual>
-        <origin xyz="0 0 0" rpy="${M_PI/2} 0 0"/>
-        <geometry>
-          <mesh filename="package://crane_x7_description/meshes/visual/joint_cover.stl"
-              scale="1 1 1"/>
-        </geometry>
-        <material name="${color_link_cover_2}"/>
+    <link name="${NAME_LINK_COVER_2_R}">
+      <visual>
+        <origin xyz="0 0 0" rpy="${M_PI/2} 0 0"/>
+        <geometry>
+          <mesh filename="package://crane_x7_description/meshes/visual/joint_cover.stl"
+              scale="1 1 1"/>
+        </geometry>
+        <material name="${COLOR_LINK_COVER_2}"/>
       </visual>
       <collision>
@@ -221,17 +173,19 @@
     </link>
     <!-- crane_x7_joint_3 -->
-    <joint name="${name_joint_3}" type="revolute">
+    <joint name="${NAME_JOINT_3}" type="revolute">
       <origin xyz="0 0 0.065" rpy="0 0 0"/>
       <axis xyz="0 0 1"/>
-      <limit effort="4.0"
-          velocity="${joint_velocity_limit}"
-          lower="${joint_3_lower_limit}"
-          upper="${joint_3_upper_limit}"/>
-      <parent link="${name_link_2}"/>
-      <child link="${name_link_3}"/>
+      <limit
+        effort="4.0"
+        velocity="${JOINT_VELOCITY_LIMIT}"
+        lower="${JOINT_3_LOWER_LIMIT}"
+        upper="${JOINT_3_UPPER_LIMIT}"
+        />
+      <parent link="${NAME_LINK_2}"/>
+      <child link="${NAME_LINK_3}"/>
       <dynamics damping="1.0e-6" friction="2.0e-1"/>
     </joint>
     <!-- crane_x7_link_3 -->
-    <link name="${name_link_3}">
+    <link name="${NAME_LINK_3}">
       <visual>
         <origin xyz="0 0 0" rpy="0 0 0"/>
@@ -240,5 +194,5 @@
               scale="1 1 1"/>
         </geometry>
-        <material name="${color_link_3}"/>
+        <material name="${COLOR_LINK_3}"/>
       </visual>
       <collision>
@@ -258,17 +212,19 @@
     </link>
     <!-- crane_x7_joint_4 -->
-    <joint name="${name_joint_4}" type="revolute">
+    <joint name="${NAME_JOINT_4}" type="revolute">
       <origin xyz="0 0 0.185" rpy="0 0 0"/>
       <axis xyz="0 -1 0"/>
-      <limit effort="4.0"
-          velocity="${joint_velocity_limit}"
-          lower="${joint_4_lower_limit}"
-          upper="${joint_4_upper_limit}"/>
-      <parent link="${name_link_3}"/>
-      <child link="${name_link_4}"/>
+      <limit
+        effort="4.0"
+        velocity="${JOINT_VELOCITY_LIMIT}"
+        lower="${JOINT_4_LOWER_LIMIT}"
+        upper="${JOINT_4_UPPER_LIMIT}"
+        />
+      <parent link="${NAME_LINK_3}"/>
+      <child link="${NAME_LINK_4}"/>
       <dynamics damping="1.0e-6" friction="2.0e-1"/>
     </joint>
     <!-- crane_x7_link_4 -->
-    <link name="${name_link_4}">
+    <link name="${NAME_LINK_4}">
       <visual>
         <origin xyz="0 0 0" rpy="${M_PI/2} 0 0"/>
@@ -277,5 +233,5 @@
               scale="1 1 1"/>
         </geometry>
-        <material name="${color_link_4}"/>
+        <material name="${COLOR_LINK_4}"/>
       </visual>
       <collision>
@@ -295,11 +251,11 @@
     </link>
     <!-- crane_x7_joint_cover_4_l -->
-    <joint name="${name_joint_cover_4_l}" type="fixed">
-      <parent link="${name_link_4}"/>
-      <child link="${name_link_cover_4_l}"/>
+    <joint name="${NAME_JOINT_COVER_4_L}" type="fixed">
+      <parent link="${NAME_LINK_4}"/>
+      <child link="${NAME_LINK_COVER_4_L}"/>
       <origin xyz="0 0.025 0" rpy="0 0 0"/>
     </joint>
     <!-- crane_x7_link_cover_4_l -->
-    <link name="${name_link_cover_4_l}">
+    <link name="${NAME_LINK_COVER_4_L}">
       <visual>
         <origin xyz="0 0 0" rpy="-${M_PI/2} 0 0"/>
@@ -308,5 +264,5 @@
               scale="1 1 1"/>
         </geometry>
-        <material name="${color_link_cover_4}"/>
+        <material name="${COLOR_LINK_COVER_4}"/>
       </visual>
       <collision>
@@ -319,18 +275,18 @@
     </link>
     <!-- crane_x7_joint_cover_4_r -->
-    <joint name="${name_joint_cover_4_r}" type="fixed">
-      <parent link="${name_link_4}"/>
-      <child link="${name_link_cover_4_r}"/>
+    <joint name="${NAME_JOINT_COVER_4_R}" type="fixed">
+      <parent link="${NAME_LINK_4}"/>
+      <child link="${NAME_LINK_COVER_4_R}"/>
       <origin xyz="0 -0.025 0" rpy="0 0 0"/>
     </joint>
     <!-- crane_x7_link_cover_4_r -->
-    <link name="${name_link_cover_4_r}">
-      <visual>
-        <origin xyz="0 0 0" rpy="${M_PI/2} 0 0"/>
-        <geometry>
-          <mesh filename="package://crane_x7_description/meshes/visual/joint_cover.stl"
-              scale="1 1 1"/>
-        </geometry>
-        <material name="${color_link_cover_4}"/>
+    <link name="${NAME_LINK_COVER_4_R}">
+      <visual>
+        <origin xyz="0 0 0" rpy="${M_PI/2} 0 0"/>
+        <geometry>
+          <mesh filename="package://crane_x7_description/meshes/visual/joint_cover.stl"
+              scale="1 1 1"/>
+        </geometry>
+        <material name="${COLOR_LINK_COVER_4}"/>
       </visual>
       <collision>
@@ -343,14 +299,19 @@
     </link>
     <!-- crane_x7_joint_5 -->
-    <joint name="${name_joint_5}" type="revolute">
+    <joint name="${NAME_JOINT_5}" type="revolute">
       <origin xyz="0 0 0.121" rpy="0 0 0"/>
       <axis xyz="0 0 1"/>
-      <limit effort="4.0" velocity="${joint_velocity_limit}" lower="${joint_5_lower_limit}" upper="${joint_5_upper_limit}"/>
-      <parent link="${name_link_4}"/>
-      <child link="${name_link_5}"/>
+      <limit
+        effort="4.0"
+        velocity="${JOINT_VELOCITY_LIMIT}"
+        lower="${JOINT_5_LOWER_LIMIT}"
+        upper="${JOINT_5_UPPER_LIMIT}"
+        />
+      <parent link="${NAME_LINK_4}"/>
+      <child link="${NAME_LINK_5}"/>
       <dynamics damping="1.0e-6" friction="2.0e-1"/>
     </joint>
     <!-- crane_x7_link_5 -->
-    <link name="${name_link_5}">
+    <link name="${NAME_LINK_5}">
       <visual>
         <origin xyz="0 0 0" rpy="0 0 0"/>
@@ -359,5 +320,5 @@
               scale="1 1 1"/>
         </geometry>
-        <material name="${color_link_5}"/>
+        <material name="${COLOR_LINK_5}"/>
       </visual>
       <collision>
@@ -377,25 +338,21 @@
     </link>
     <!-- logo -->
-    <xacro:crane_x7_logos
-      parent="${name_link_5}"
-      name_link_logo_symbol_l="${name_link_logo_symbol_l}"
-      name_link_logo_symbol_r="${name_link_logo_symbol_r}"
-      name_link_logo_text_l="${name_link_logo_text_l}"
-      name_link_logo_text_r="${name_link_logo_text_r}"
-      name_joint_logo_symbol_l="${name_joint_logo_symbol_l}"
-      name_joint_logo_symbol_r="${name_joint_logo_symbol_r}"
-      name_joint_logo_text_l="${name_joint_logo_text_l}"
-      name_joint_logo_text_r="${name_joint_logo_text_r}"/>
+    <xacro:crane_x7_logos parent="${NAME_LINK_5}"/>
     <!-- crane_x7_joint_6 -->
-    <joint name="${name_joint_6}" type="revolute">
+    <joint name="${NAME_JOINT_6}" type="revolute">
       <origin xyz="0 0 0.129" rpy="0 0 0"/>
       <axis xyz="0 -1 0"/>
-      <limit effort="4.0" velocity="${joint_velocity_limit}" lower="${joint_6_lower_limit}" upper="${joint_6_upper_limit}"/>
-      <parent link="${name_link_5}"/>
-      <child link="${name_link_6}"/>
+      <limit
+        effort="4.0"
+        velocity="${JOINT_VELOCITY_LIMIT}"
+        lower="${JOINT_6_LOWER_LIMIT}"
+        upper="${JOINT_6_UPPER_LIMIT}"
+        />
+      <parent link="${NAME_LINK_5}"/>
+      <child link="${NAME_LINK_6}"/>
       <dynamics damping="1.0e-6" friction="2.0e-1"/>
     </joint>
     <!-- crane_x7_link_6 -->
-    <link name="${name_link_6}">
+    <link name="${NAME_LINK_6}">
       <visual>
         <origin xyz="0 0 0" rpy="${M_PI/2} 0 0"/>
@@ -404,5 +361,5 @@
               scale="1 1 1"/>
         </geometry>
-        <material name="${color_link_6}"/>
+        <material name="${COLOR_LINK_6}"/>
       </visual>
       <collision>
@@ -422,10 +379,15 @@
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
File: urdf/crane_x7_mounting_plate.xacro (robot description, xacro)
@@ -5,16 +5,11 @@
   <xacro:property name="SCALE_CM" value="0.01"/>
   <xacro:property name="MOUNTING_PLATE_THICKNESS" value="0.005"/>
-  <xacro:macro name="crane_x7_mounting_plate"
-      params="parent
-              name_link_mounting_plate
-              name_joint_mounting_plate
-              color
-              *origin">
-    <joint name="${name_joint_mounting_plate}" type="fixed">
+  <xacro:macro name="crane_x7_mounting_plate" params="parent color *origin">
+    <joint name="${NAME_JOINT_MOUNTING_PLATE}" type="fixed">
       <xacro:insert_block name="origin"/>
       <parent link="${parent}"/>
-      <child link="${name_link_mounting_plate}"/>
+      <child link="${NAME_LINK_MOUNTING_PLATE}"/>
     </joint>
-    <link name="${name_link_mounting_plate}">
+    <link name="${NAME_LINK_MOUNTING_PLATE}">
       <visual>
         <origin xyz="0 0 0" rpy="0 0 0"/>

File: urdf/crane_x7_rt_logos.xacro (robot description, xacro)
@@ -1,16 +1,7 @@
 <?xml version="1.0"?>
 <robot xmlns:xacro="http://ros.org/wiki/xacro">
-  <xacro:macro name="crane_x7_logos"
-      params="parent
-              name_link_logo_symbol_l
-              name_link_logo_symbol_r
-              name_link_logo_text_l
-              name_link_logo_text_r
-              name_joint_logo_symbol_l
-              name_joint_logo_symbol_r
-              name_joint_logo_text_l
-              name_joint_logo_text_r">
+  <xacro:macro name="crane_x7_logos" params="parent">
     <!-- Left side logo text -->
-    <link name="${name_link_logo_text_l}">
+    <link name="${NAME_LINK_LOGO_TEXT_L}">
       <visual>
         <origin xyz="0 0 0" rpy="-${M_PI/2} ${M_PI/2} 0"/>
@@ -29,11 +20,11 @@
       </collision>
     </link>
-    <joint name="${name_joint_logo_text_l}" type="fixed">
+    <joint name="${NAME_JOINT_LOGO_TEXT_L}" type="fixed">
       <parent link="${parent}"/>
-      <child link="${name_link_logo_text_l}"/>
+      <child link="${NAME_LINK_LOGO_TEXT_L}"/>
       <origin xyz="0 0.0345 0.095" rpy="0 0 0"/>
     </joint>
     <!-- Left side logo symbol -->
-    <link name="${name_link_logo_symbol_l}">
+    <link name="${NAME_LINK_LOGO_SYMBOL_L}">
       <visual>
         <origin xyz="0 0 0" rpy="-${M_PI/2} ${M_PI/2} 0"/>
@@ -52,11 +43,11 @@
       </collision>
     </link>
-    <joint name="${name_joint_logo_symbol_l}" type="fixed">
+    <joint name="${NAME_JOINT_LOGO_SYMBOL_L}" type="fixed">
       <parent link="${parent}"/>
-      <child link="${name_link_logo_symbol_l}"/>
+      <child link="${NAME_LINK_LOGO_SYMBOL_L}"/>
       <origin xyz="0 0.0345 0.132" rpy="0 0 0"/>
     </joint>
     <!-- Right side logo text -->
-    <link name="${name_link_logo_text_r}">
+    <link name="${NAME_LINK_LOGO_TEXT_R}">
       <visual>
         <origin xyz="0 0 0" rpy="${M_PI/2} -${M_PI/2} 0"/>
@@ -75,11 +66,11 @@
       </collision>
     </link>
-    <joint name="${name_joint_logo_text_r}" type="fixed">
+    <joint name="${NAME_JOINT_LOGO_TEXT_R}" type="fixed">
       <parent link="${parent}"/>
-      <child link="${name_link_logo_text_r}"/>
+      <child link="${NAME_LINK_LOGO_TEXT_R}"/>
       <origin xyz="0 -0.0345 0.104" rpy="0 0 0"/>
     </joint>
     <!-- Right side logo symbol -->
-    <link name="${name_link_logo_symbol_r}">
+    <link name="${NAME_LINK_LOGO_SYMBOL_R}">
       <visual>
         <origin xyz="0 0 0" rpy="${M_PI/2} -${M_PI/2} 0"/>
@@ -98,7 +89,7 @@
       </collision>
     </link>
-    <joint name="${name_joint_logo_symbol_r}" type="fixed">
+    <joint name="${NAME_JOINT_LOGO_SYMBOL_R}" type="fixed">
       <parent link="${parent}"/>
-      <child link="${name_link_logo_symbol_r}"/>
+      <child link="${NAME_LINK_LOGO_SYMBOL_R}"/>
       <origin xyz="0 -0.0345 0.065" rpy="0 0 0"/>
     </joint>

File: urdf/crane_x7_wide_two_finger_gripper.xacro (robot description, xacro)
@@ -4,15 +4,6 @@
   <xacro:property name="SCALE_MM" value="0.001"/>
   <xacro:property name="SCALE_CM" value="0.01"/>
-  <xacro:macro name="crane_x7_wide_two_finger_gripper"
-    params="name_link_gripper_base
-            name_link_gripper_finger_a
-            name_link_gripper_finger_b
-            name_joint_gripper_finger_a
-            name_joint_gripper_finger_b
-            color
-            joint_velocity_limit
-            joint_hand_lower_limit
-            joint_hand_upper_limit">
-    <link name="${name_link_gripper_base}">
+  <xacro:macro name="crane_x7_wide_two_finger_gripper">
+    <link name="${NAME_LINK_GRIPPER_BASE}">
       <visual>
         <origin xyz="0 0 0" rpy="0 0 0"/>
@@ -21,5 +12,5 @@
               scale="1 1 1"/>
         </geometry>
-        <material name="${color}"/>
+        <material name="${COLOR_HAND}"/>
       </visual>
       <collision>
@@ -38,13 +29,17 @@
       </inertial>
     </link>
-    <joint name="${name_joint_gripper_finger_a}" type="revolute">
+    <joint name="${NAME_JOINT_GRIPPER_FINGER_A}" type="revolute">
       <origin xyz="-0.012 0.0 0.024" rpy="0 0 0"/>
       <axis xyz="0 -1 0"/>
-      <limit effort="4.0" velocity="${joint_velocity_limit}" lower="${joint_hand_lower_limit}" upper="${joint_hand_upper_limit}"/>
-      <parent link="${name_link_gripper_base}"/>
-      <child link="${name_link_gripper_finger_a}"/>
+      <limit
+        effort="4.0"
+        velocity="${JOINT_VELOCITY_LIMIT}"
+        lower="${JOINT_HAND_LOWER_LIMIT}"
+        upper="${JOINT_HAND_UPPER_LIMIT}"/>
+      <parent link="${NAME_LINK_GRIPPER_BASE}"/>
+      <child link="${NAME_LINK_GRIPPER_FINGER_A}"/>
       <dynamics damping="1.0e-6" friction="8.0e-1"/>
     </joint>
-    <link name="${name_link_gripper_finger_a}">
+    <link name="${NAME_LINK_GRIPPER_FINGER_A}">
       <visual>
         <origin xyz="0 0 0" rpy="${M_PI/2} 0 0"/>
@@ -53,5 +48,5 @@
               scale="1 1 1"/>
         </geometry>
-        <material name="${color}"/>
+        <material name="${COLOR_HAND}"/>
       </visual>
       <collision>
@@ -73,19 +68,24 @@
     See https://github.com/ros-controls/gazebo_ros2_control/issues/173
     -->
-    <joint name="${name_joint_gripper_finger_b}_mimic" type="fixed">
+    <joint name="${NAME_JOINT_GRIPPER_FINGER_B}_mimic" type="fixed">
       <parent link="world" />
       <child link="dummy_mimic_fix" />
     </joint>
     <link name="dummy_mimic_fix"/>
-    <joint name="${name_joint_gripper_finger_b}" type="revolute">
+    <joint name="${NAME_JOINT_GRIPPER_FINGER_B}" type="revolute">
       <origin xyz="0.012 0.0 0.024" rpy="0 0 0"/>
       <axis xyz="0 1 0"/>
-      <limit effort="4.0" velocity="${joint_velocity_limit}" lower="${joint_hand_lower_limit}" upper="${joint_hand_upper_limit}"/>
-      <parent link="${name_link_gripper_base}"/>
-      <child link="${name_link_gripper_finger_b}"/>
-      <mimic joint="${name_joint_gripper_finger_a}"/>
+      <limit
+        effort="4.0"
+        velocity="${JOINT_VELOCITY_LIMIT}"
+        lower="${JOINT_HAND_LOWER_LIMIT}"
+        upper="${JOINT_HAND_UPPER_LIMIT}"
+        />
+      <parent link="${NAME_LINK_GRIPPER_BASE}"/>
+      <child link="${NAME_LINK_GRIPPER_FINGER_B}"/>
+      <mimic joint="${NAME_JOINT_GRIPPER_FINGER_A}"/>
       <dynamics damping="1.0e-6" friction="8.0e-1"/>
     </joint>
-    <link name="${name_link_gripper_finger_b}">
+    <link name="${NAME_LINK_GRIPPER_FINGER_B}">
       <visual>
         <origin xyz="0 0 0" rpy="${M_PI/2} 0 0"/>
@@ -94,5 +94,5 @@
               scale="1 1 1"/>
         </geometry>
-        <material name="${color}"/>
+        <material name="${COLOR_HAND}"/>
       </visual>
       <collision>
