Commit message: マテリアルの定義場所をS17に合わせる

File: urdf/crane_x7.urdf.xacro (robot description, xacro)
@@ -25,4 +25,22 @@
   <xacro:property name="GZ_CONTROL_CONFIG_PACKAGE" value="$(arg gz_control_config_package)"/>
   <xacro:property name="GZ_CONTROL_CONFIG_FILE_PATH" value="$(arg gz_control_config_file_path)"/>
+  <material name="black">
+    <color rgba="0.2 0.2 0.2 1.0"/>
+  </material>
+  <material name="white">
+    <color rgba="0.95 0.95 0.95 1.0"/>
+  </material>
+  <material name="silver">
+    <color rgba="0.75 0.75 0.75 1.0"/>
+  </material>
+  <material name="red">
+    <color rgba="1.0 0.3 0.3 1.0"/>
+  </material>
+  <material name="green">
+    <color rgba="0.3 1.0 0.3 1.0"/>
+  </material>
+  <material name="blue">
+    <color rgba="0.3 0.3 1.0 1.0"/>
+  </material>
   <xacro:property name="M_PI" value="3.14159"/>
   <xacro:property name="NAME_LINK_MOUNTING_PLATE" value="crane_x7_mounting_plate_link"/>

File: urdf/crane_x7.xacro (robot description, xacro)
@@ -5,22 +5,4 @@
   <xacro:include filename="$(find crane_x7_description)/urdf/crane_x7_wide_two_finger_gripper.xacro"/>
   <xacro:include filename="$(find crane_x7_description)/urdf/crane_x7_rt_logos.xacro"/>
-  <material name="black">
-    <color rgba="0.2 0.2 0.2 1.0"/>
-  </material>
-  <material name="white">
-    <color rgba="0.95 0.95 0.95 1.0"/>
-  </material>
-  <material name="silver">
-    <color rgba="0.75 0.75 0.75 1.0"/>
-  </material>
-  <material name="red">
-    <color rgba="1.0 0.3 0.3 1.0"/>
-  </material>
-  <material name="green">
-    <color rgba="0.3 1.0 0.3 1.0"/>
-  </material>
-  <material name="blue">
-    <color rgba="0.3 0.3 1.0 1.0"/>
-  </material>
   <xacro:macro name="crane_x7" params="parent *origin">
     <!-- Mounting plate

Commit message: 円周率の定数を削除してradians()に置き換える

File: urdf/crane_x7.urdf.xacro (robot description, xacro)
@@ -43,5 +43,4 @@
     <color rgba="0.3 0.3 1.0 1.0"/>
   </material>
-  <xacro:property name="M_PI" value="3.14159"/>
   <xacro:property name="NAME_LINK_MOUNTING_PLATE" value="crane_x7_mounting_plate_link"/>
   <xacro:property name="NAME_LINK_BASE" value="crane_x7_shoulder_fixed_part_link"/>

File: urdf/crane_x7_arm.xacro (robot description, xacro)
@@ -51,5 +51,5 @@
     <link name="${NAME_LINK_1}">
       <visual>
-        <origin xyz="0 0 0" rpy="0 0 ${M_PI}"/>
+        <origin xyz="0 0 0" rpy="0 0 ${radians(180)}"/>
         <geometry>
           <mesh filename="package://crane_x7_description/meshes/visual/base_revolute_part.stl"
@@ -59,5 +59,5 @@
       </visual>
       <collision>
-        <!--<origin xyz="0 0 0" rpy="0 0 ${M_PI}"/>-->
+        <!--<origin xyz="0 0 0" rpy="0 0 ${radians(180)}"/>-->
         <!--<geometry>-->
           <!--<mesh filename="package://crane_x7_description/meshes/collision/base_revolute_part.stl"-->
@@ -70,5 +70,5 @@
       </collision>
       <collision>
-        <origin xyz="0 0 0.064" rpy="${M_PI/2} 0 0"/>
+        <origin xyz="0 0 0.064" rpy="${radians(90)} 0 0"/>
         <geometry>
           <cylinder radius="0.034" length="0.0491"/>
@@ -100,5 +100,5 @@
     <link name="${NAME_LINK_2}">
       <visual>
-        <origin xyz="0 0 0" rpy="${M_PI/2} 0 0"/>
+        <origin xyz="0 0 0" rpy="${radians(90)} 0 0"/>
         <geometry>
           <mesh filename="package://crane_x7_description/meshes/visual/rotating_link_type_1_fixed_part.stl"
@@ -108,5 +108,5 @@
       </visual>
       <collision>
-        <origin xyz="0 0 0" rpy="${M_PI/2} 0 0"/>
+        <origin xyz="0 0 0" rpy="${radians(90)} 0 0"/>
         <geometry>
           <mesh filename="package://crane_x7_description/meshes/collision/rotating_link_type_1_fixed_part.stl"
@@ -116,5 +116,5 @@
       <inertial>
         <mass value="0.136"/>
-        <origin xyz="3.10E-05 1.90E-05 3.42E-02" rpy="${M_PI/2} 0 0"/>
+        <origin xyz="3.10E-05 1.90E-05 3.42E-02" rpy="${radians(90)} 0 0"/>
         <inertia ixx="1.68E-04" ixy="2.05E-08" ixz="-4.00E-07"
           iyy="9.62E-05" iyz="6.24E-08"
@@ -131,5 +131,5 @@
     <link name="${NAME_LINK_COVER_2_L}">
       <visual>
-        <origin xyz="0 0 0" rpy="-${M_PI/2} 0 0"/>
+        <origin xyz="0 0 0" rpy="${radians(-90)} 0 0"/>
         <geometry>
           <mesh filename="package://crane_x7_description/meshes/visual/joint_cover.stl"
@@ -139,5 +139,5 @@
       </visual>
       <collision>
-        <origin xyz="0 0 0" rpy="-${M_PI/2} 0 0"/>
+        <origin xyz="0 0 0" rpy="${radians(-90)} 0 0"/>
         <geometry>
           <mesh filename="package://crane_x7_description/meshes/visual/joint_cover.stl"
@@ -155,5 +155,5 @@
     <link name="${NAME_LINK_COVER_2_R}">
       <visual>
-        <origin xyz="0 0 0" rpy="${M_PI/2} 0 0"/>
+        <origin xyz="0 0 0" rpy="${radians(90)} 0 0"/>
         <geometry>
           <mesh filename="package://crane_x7_description/meshes/visual/joint_cover.stl"
@@ -163,5 +163,5 @@
       </visual>
       <collision>
-        <origin xyz="0 0 0" rpy="${M_PI/2} 0 0"/>
+        <origin xyz="0 0 0" rpy="${radians(90)} 0 0"/>
         <geometry>
           <mesh filename="package://crane_x7_description/meshes/visual/joint_cover.stl"
@@ -226,5 +226,5 @@
     <link name="${NAME_LINK_4}">
       <visual>
-        <origin xyz="0 0 0" rpy="${M_PI/2} 0 0"/>
+        <origin xyz="0 0 0" rpy="${radians(90)} 0 0"/>
         <geometry>
           <mesh filename="package://crane_x7_description/meshes/visual/rotating_link_type_2_fixed_part.stl"
@@ -234,5 +234,5 @@
       </visual>
       <collision>
-        <origin xyz="0 0 0" rpy="${M_PI/2} 0 0"/>
+        <origin xyz="0 0 0" rpy="${radians(90)} 0 0"/>
         <geometry>
           <mesh filename="package://crane_x7_description/meshes/collision/rotating_link_type_2_fixed_part.stl"
@@ -242,5 +242,5 @@
       <inertial>
         <mass value="0.222"/>
-        <origin xyz="-9.39E-03 6.40E-05 8.04E-02" rpy="${M_PI/2} 0 0"/>
+        <origin xyz="-9.39E-03 6.40E-05 8.04E-02" rpy="${radians(90)} 0 0"/>
         <inertia ixx="4.89E-04" ixy="-3.90E-06" ixz="8.29E-08"
           iyy="1.14E-04" iyz="2.82E-06"
@@ -257,5 +257,5 @@
     <link name="${NAME_LINK_COVER_4_L}">
       <visual>
-        <origin xyz="0 0 0" rpy="-${M_PI/2} 0 0"/>
+        <origin xyz="0 0 0" rpy="${radians(-90)} 0 0"/>
         <geometry>
           <mesh filename="package://crane_x7_description/meshes/visual/joint_cover.stl"
@@ -265,5 +265,5 @@
       </visual>
       <collision>
-        <origin xyz="0 0 0" rpy="-${M_PI/2} 0 0"/>
+        <origin xyz="0 0 0" rpy="${radians(-90)} 0 0"/>
         <geometry>
           <mesh filename="package://crane_x7_description/meshes/visual/joint_cover.stl"
@@ -281,5 +281,5 @@
     <link name="${NAME_LINK_COVER_4_R}">
       <visual>
-        <origin xyz="0 0 0" rpy="${M_PI/2} 0 0"/>
+        <origin xyz="0 0 0" rpy="${radians(90)} 0 0"/>
         <geometry>
           <mesh filename="package://crane_x7_description/meshes/visual/joint_cover.stl"
@@ -289,5 +289,5 @@
       </visual>
       <collision>
-        <origin xyz="0 0 0" rpy="${M_PI/2} 0 0"/>
+        <origin xyz="0 0 0" rpy="${radians(90)} 0 0"/>
         <geometry>
           <mesh filename="package://crane_x7_description/meshes/visual/joint_cover.stl"
@@ -354,5 +354,5 @@
     <link name="${NAME_LINK_6}">
       <visual>
-        <origin xyz="0 0 0" rpy="${M_PI/2} 0 0"/>
+        <origin xyz="0 0 0" rpy="${radians(90)} 0 0"/>
         <geometry>
           <mesh filename="package://crane_x7_description/meshes/visual/wrist.stl"
@@ -362,5 +362,5 @@
       </visual>
       <collision>
-        <origin xyz="0 0 0" rpy="${M_PI/2} 0 0"/>
+        <origin xyz="0 0 0" rpy="${radians(90)} 0 0"/>
         <geometry>
           <mesh filename="package://crane_x7_description/meshes/collision/wrist.stl"
@@ -370,5 +370,5 @@
       <inertial>
         <mass value="0.14"/>
-        <origin xyz="6.10E-03 8.26E-04 -3.55E-03" rpy="${M_PI/2} 0 0"/>
+        <origin xyz="6.10E-03 8.26E-04 -3.55E-03" rpy="${radians(90)} 0 0"/>
         <inertia ixx="4.01E-05" ixy="-2.91E-06" ixz="6.39E-07"
           iyy="6.13E-05" iyz="-4.90E-07"

File: urdf/crane_x7_rt_logos.xacro (robot description, xacro)
@@ -5,5 +5,5 @@
     <link name="${NAME_LINK_LOGO_TEXT_L}">
       <visual>
-        <origin xyz="0 0 0" rpy="-${M_PI/2} ${M_PI/2} 0"/>
+        <origin xyz="0 0 0" rpy="${radians(-90)} ${radians(90)} 0"/>
         <geometry>
           <mesh filename="package://crane_x7_description/meshes/visual/rtcorp_logo_name.stl"
@@ -13,5 +13,5 @@
       </visual>
       <collision>
-        <origin xyz="0 0 0" rpy="-${M_PI/2} ${M_PI/2} 0"/>
+        <origin xyz="0 0 0" rpy="${radians(-90)} ${radians(90)} 0"/>
         <geometry>
           <mesh filename="package://crane_x7_description/meshes/visual/rtcorp_logo_name.stl"
@@ -28,5 +28,5 @@
     <link name="${NAME_LINK_LOGO_SYMBOL_L}">
       <visual>
-        <origin xyz="0 0 0" rpy="-${M_PI/2} ${M_PI/2} 0"/>
+        <origin xyz="0 0 0" rpy="${radians(-90)} ${radians(90)} 0"/>
         <geometry>
           <mesh filename="package://crane_x7_description/meshes/visual/rtcorp_logo_rabbit.stl"
@@ -36,5 +36,5 @@
       </visual>
       <collision>
-        <origin xyz="0 0 0" rpy="-${M_PI/2} ${M_PI/2} 0"/>
+        <origin xyz="0 0 0" rpy="${radians(-90)} ${radians(90)} 0"/>
         <geometry>
           <mesh filename="package://crane_x7_description/meshes/visual/rtcorp_logo_rabbit.stl"
@@ -51,5 +51,5 @@
     <link name="${NAME_LINK_LOGO_TEXT_R}">
       <visual>
-        <origin xyz="0 0 0" rpy="${M_PI/2} -${M_PI/2} 0"/>
+        <origin xyz="0 0 0" rpy="${radians(90)} ${radians(-90)} 0"/>
         <geometry>
           <mesh filename="package://crane_x7_description/meshes/visual/rtcorp_logo_name.stl"
@@ -59,5 +59,5 @@
       </visual>
       <collision>
-        <origin xyz="0 0 0" rpy="${M_PI/2} -${M_PI/2} 0"/>
+        <origin xyz="0 0 0" rpy="${radians(90)} ${radians(-90)} 0"/>
         <geometry>
           <mesh filename="package://crane_x7_description/meshes/visual/rtcorp_logo_name.stl"
@@ -74,5 +74,5 @@
     <link name="${NAME_LINK_LOGO_SYMBOL_R}">
       <visual>
-        <origin xyz="0 0 0" rpy="${M_PI/2} -${M_PI/2} 0"/>
+        <origin xyz="0 0 0" rpy="${radians(90)} ${radians(-90)} 0"/>
         <geometry>
           <mesh filename="package://crane_x7_description/meshes/visual/rtcorp_logo_rabbit.stl"
@@ -82,5 +82,5 @@
       </visual>
       <collision>
-        <origin xyz="0 0 0" rpy="${M_PI/2} -${M_PI/2} 0"/>
+        <origin xyz="0 0 0" rpy="${radians(90)} ${radians(-90)} 0"/>
         <geometry>
           <mesh filename="package://crane_x7_description/meshes/visual/rtcorp_logo_rabbit.stl"

File: urdf/crane_x7_wide_two_finger_gripper.xacro (robot description, xacro)
@@ -40,5 +40,5 @@
     <link name="${NAME_LINK_GRIPPER_FINGER_A}">
       <visual>
-        <origin xyz="0 0 0" rpy="${M_PI/2} 0 0"/>
+        <origin xyz="0 0 0" rpy="${radians(90)} 0 0"/>
         <geometry>
           <mesh filename="package://crane_x7_description/meshes/visual/wide_two_finger_gripper_finger_a.stl"
@@ -48,5 +48,5 @@
       </visual>
       <collision>
-        <origin xyz="0 0 0" rpy="${M_PI/2} 0 0"/>
+        <origin xyz="0 0 0" rpy="${radians(90)} 0 0"/>
         <geometry>
           <mesh filename="package://crane_x7_description/meshes/collision/wide_two_finger_gripper_finger_a.stl"
@@ -56,5 +56,5 @@
       <inertial>
         <mass value="0.0158"/>
-        <origin xyz="-2.65E-03 3.54E-03 2.69E-02" rpy="${M_PI/2} 0 0"/>
+        <origin xyz="-2.65E-03 3.54E-03 2.69E-02" rpy="${radians(90)} 0 0"/>
         <inertia ixx="1.01E-05" ixy="-1.97E-07" ixz="-9.89E-08"
         iyy="4.95E-06" iyz="5.37E-07"
@@ -86,5 +86,5 @@
     <link name="${NAME_LINK_GRIPPER_FINGER_B}">
       <visual>
-        <origin xyz="0 0 0" rpy="${M_PI/2} 0 0"/>
+        <origin xyz="0 0 0" rpy="${radians(90)} 0 0"/>
         <geometry>
           <mesh filename="package://crane_x7_description/meshes/visual/wide_two_finger_gripper_finger_b.stl"
@@ -94,5 +94,5 @@
       </visual>
       <collision>
-        <origin xyz="0 0 0" rpy="${M_PI/2} 0 0"/>
+        <origin xyz="0 0 0" rpy="${radians(90)} 0 0"/>
         <geometry>
           <mesh filename="package://crane_x7_description/meshes/collision/wide_two_finger_gripper_finger_b.stl"
@@ -102,5 +102,5 @@
       <inertial>
         <mass value="0.0139"/>
-        <origin xyz="3.01E-03 2.85E-03 3.09E-02" rpy="${M_PI/2} 0 0"/>
+        <origin xyz="3.01E-03 2.85E-03 3.09E-02" rpy="${radians(90)} 0 0"/>
         <inertia ixx="7.48E-06" ixy="3.61E-07" ixz="6.34E-08"
         iyy="4.09E-06" iyz="2.28E-07"
