Commit message: 色のpropertyを廃止

File: urdf/crane_x7.urdf.xacro (robot description, xacro)
@@ -30,14 +30,4 @@
   </joint>
   <xacro:property name="M_PI" value="3.14159"/>
-  <xacro:property name="COLOR_LINK_BASE" value="red"/>
-  <xacro:property name="COLOR_LINK_1" value="white"/>
-  <xacro:property name="COLOR_LINK_COVER_2" value="red"/>
-  <xacro:property name="COLOR_LINK_2" value="white"/>
-  <xacro:property name="COLOR_LINK_3" value="white"/>
-  <xacro:property name="COLOR_LINK_COVER_4" value="red"/>
-  <xacro:property name="COLOR_LINK_4" value="white"/>
-  <xacro:property name="COLOR_LINK_5" value="white"/>
-  <xacro:property name="COLOR_LINK_6" value="white"/>
-  <xacro:property name="COLOR_HAND" value="red"/>
   <xacro:property name="JOINT_VELOCITY_LIMIT" value="4.81710873"/>
   <xacro:property name="JOINT_1_LOWER_LIMIT" value="${radians(-157)}"/>
@@ -66,14 +56,4 @@
   <xacro:crane_x7
     parent="base_link"
-    color_link_base="${COLOR_LINK_BASE}"
-    color_link_1="${COLOR_LINK_1}"
-    color_link_cover_2="${COLOR_LINK_COVER_2}"
-    color_link_2="${COLOR_LINK_2}"
-    color_link_3="${COLOR_LINK_3}"
-    color_link_cover_4="${COLOR_LINK_COVER_4}"
-    color_link_4="${COLOR_LINK_4}"
-    color_link_5="${COLOR_LINK_5}"
-    color_link_6="${COLOR_LINK_6}"
-    color_hand="${COLOR_HAND}"
     joint_velocity_limit="${JOINT_VELOCITY_LIMIT}"
     joint_1_lower_limit="${JOINT_1_LOWER_LIMIT}"

File: urdf/crane_x7.xacro (robot description, xacro)
@@ -25,14 +25,4 @@
   <xacro:macro name="crane_x7"
       params="parent
-              color_link_base
-              color_link_1
-              color_link_cover_2
-              color_link_2
-              color_link_3
-              color_link_cover_4
-              color_link_4
-              color_link_5
-              color_link_6
-              color_hand
               joint_velocity_limit
               joint_1_lower_limit
@@ -57,6 +47,5 @@
          (Root of the manipulator's TF tree) -->
     <xacro:crane_x7_mounting_plate
-        parent="${parent}"
-        color="black">
+      parent="${parent}">
       <xacro:insert_block name="origin"/>
     </xacro:crane_x7_mounting_plate>
@@ -64,13 +53,4 @@
     <xacro:crane_x7_arm
       parent="crane_x7_mounting_plate_link"
-        color_link_base="${color_link_base}"
-        color_link_1="${color_link_1}"
-        color_link_cover_2="${color_link_cover_2}"
-        color_link_2="${color_link_2}"
-        color_link_3="${color_link_3}"
-        color_link_cover_4="${color_link_cover_4}"
-        color_link_4="${color_link_4}"
-        color_link_5="${color_link_5}"
-        color_link_6="${color_link_6}"
         joint_velocity_limit="${joint_velocity_limit}"
         joint_1_lower_limit="${joint_1_lower_limit}"
@@ -103,5 +83,4 @@
     <!-- End effector -->
     <xacro:crane_x7_wide_two_finger_gripper
-        color="${color_hand}"
         joint_velocity_limit="${joint_velocity_limit}"
         joint_hand_lower_limit="${joint_hand_lower_limit}"

File: urdf/crane_x7_arm.xacro (robot description, xacro)
@@ -6,13 +6,4 @@
   <xacro:macro name="crane_x7_arm"
       params="parent
-              color_link_base
-              color_link_1
-              color_link_cover_2
-              color_link_2
-              color_link_3
-              color_link_cover_4
-              color_link_4
-              color_link_5
-              color_link_6
               joint_velocity_limit
               joint_1_lower_limit
@@ -45,5 +36,5 @@
               scale="1 1 1"/>
         </geometry>
-        <material name="${color_link_base}"/>
+        <material name="red"/>
       </visual>
       <collision>
@@ -79,5 +70,5 @@
               scale="1 1 1"/>
         </geometry>
-        <material name="${color_link_1}"/>
+        <material name="white"/>
       </visual>
       <collision>
@@ -123,5 +114,5 @@
               scale="1 1 1"/>
         </geometry>
-        <material name="${color_link_2}"/>
+        <material name="white"/>
       </visual>
       <collision>
@@ -154,5 +145,5 @@
               scale="1 1 1"/>
         </geometry>
-        <material name="${color_link_cover_2}"/>
+        <material name="red"/>
       </visual>
       <collision>
@@ -178,5 +169,5 @@
               scale="1 1 1"/>
         </geometry>
-        <material name="${color_link_cover_2}"/>
+        <material name="red"/>
       </visual>
       <collision>
@@ -208,5 +199,5 @@
               scale="1 1 1"/>
         </geometry>
-        <material name="${color_link_3}"/>
+        <material name="white"/>
       </visual>
       <collision>
@@ -245,5 +236,5 @@
               scale="1 1 1"/>
         </geometry>
-        <material name="${color_link_4}"/>
+        <material name="white"/>
       </visual>
       <collision>
@@ -276,5 +267,5 @@
               scale="1 1 1"/>
         </geometry>
-        <material name="${color_link_cover_4}"/>
+        <material name="red"/>
       </visual>
       <collision>
@@ -300,5 +291,5 @@
               scale="1 1 1"/>
         </geometry>
-        <material name="${color_link_cover_4}"/>
+        <material name="red"/>
       </visual>
       <collision>
@@ -327,5 +318,5 @@
               scale="1 1 1"/>
         </geometry>
-        <material name="${color_link_5}"/>
+        <material name="white"/>
       </visual>
       <collision>
@@ -364,5 +355,5 @@
               scale="1 1 1"/>
         </geometry>
-        <material name="${color_link_6}"/>
+        <material name="white"/>
       </visual>
       <collision>

File: urdf/crane_x7_mounting_plate.xacro (robot description, xacro)
@@ -7,5 +7,4 @@
   <xacro:macro name="crane_x7_mounting_plate"
       params="parent
-              color
               *origin">
     <joint name="crane_x7_mounting_plate_joint" type="fixed">
@@ -21,5 +20,5 @@
               scale="1 1 1"/>
         </geometry>
-        <material name="${color}"/>
+        <material name="black"/>
       </visual>
       <collision>

File: urdf/crane_x7_wide_two_finger_gripper.xacro (robot description, xacro)
@@ -5,6 +5,5 @@
   <xacro:property name="SCALE_CM" value="0.01"/>
   <xacro:macro name="crane_x7_wide_two_finger_gripper"
-    params="color
-            joint_velocity_limit
+    params="joint_velocity_limit
             joint_hand_lower_limit
             joint_hand_upper_limit">
@@ -16,5 +15,5 @@
               scale="1 1 1"/>
         </geometry>
-        <material name="${color}"/>
+        <material name="red"/>
       </visual>
       <collision>
@@ -48,5 +47,5 @@
               scale="1 1 1"/>
         </geometry>
-        <material name="${color}"/>
+        <material name="red"/>
       </visual>
       <collision>
@@ -81,5 +80,5 @@
               scale="1 1 1"/>
         </geometry>
-        <material name="${color}"/>
+        <material name="red"/>
       </visual>
       <collision>

Commit message: 不要なpropertyを廃止 (#19)
* リンクとジョイントのpropertyを廃止

* 色のpropertyを廃止

File: urdf/crane_x7.urdf.xacro (robot description, xacro)
@@ -30,53 +30,4 @@
   </joint>
   <xacro:property name="M_PI" value="3.14159"/>
-  <xacro:property name="NAME_LINK_MOUNTING_PLATE" value="crane_x7_mounting_plate_link"/>
-  <xacro:property name="NAME_LINK_BASE" value="crane_x7_shoulder_fixed_part_link"/>
-  <xacro:property name="NAME_LINK_1" value="crane_x7_shoulder_revolute_part_link"/>
-  <xacro:property name="NAME_LINK_2" value="crane_x7_upper_arm_fixed_part_link"/>
-  <xacro:property name="NAME_LINK_3" value="crane_x7_upper_arm_revolute_part_link"/>
-  <xacro:property name="NAME_LINK_4" value="crane_x7_lower_arm_fixed_part_link"/>
-  <xacro:property name="NAME_LINK_5" value="crane_x7_lower_arm_revolute_part_link"/>
-  <xacro:property name="NAME_LINK_6" value="crane_x7_wrist_link"/>
-  <xacro:property name="NAME_LINK_7" value="crane_x7_gripper_base_link"/>
-  <xacro:property name="NAME_LINK_COVER_2_L" value="crane_x7_upper_arm_fixed_part_joint_cover_l_link"/>
-  <xacro:property name="NAME_LINK_COVER_2_R" value="crane_x7_upper_arm_fixed_part_joint_cover_r_link"/>
-  <xacro:property name="NAME_LINK_COVER_4_L" value="crane_x7_lower_arm_fixed_part_joint_cover_l_link"/>
-  <xacro:property name="NAME_LINK_COVER_4_R" value="crane_x7_lower_arm_fixed_part_joint_cover_r_link"/>
-  <xacro:property name="NAME_LINK_LOGO_SYMBOL_L" value="crane_x7_lower_arm_revolute_part_logo_symbol_l_link"/>
-  <xacro:property name="NAME_LINK_LOGO_SYMBOL_R" value="crane_x7_lower_arm_revolute_part_logo_symbol_r_link"/>
-  <xacro:property name="NAME_LINK_LOGO_TEXT_L" value="crane_x7_lower_arm_revolute_part_logo_text_l_link"/>
-  <xacro:property name="NAME_LINK_LOGO_TEXT_R" value="crane_x7_lower_arm_revolute_part_logo_text_r_link"/>
-  <xacro:property name="NAME_LINK_GRIPPER_BASE" value="crane_x7_gripper_base_link"/>
-  <xacro:property name="NAME_LINK_GRIPPER_FINGER_A" value="crane_x7_gripper_finger_a_link"/>
-  <xacro:property name="NAME_LINK_GRIPPER_FINGER_B" value="crane_x7_gripper_finger_b_link"/>
-  <xacro:property name="NAME_JOINT_MOUNTING_PLATE" value="crane_x7_mounting_plate_joint"/>
-  <xacro:property name="NAME_JOINT_BASE" value="crane_x7_shoulder_fixed_part_mount_joint"/>
-  <xacro:property name="NAME_JOINT_1" value="crane_x7_shoulder_fixed_part_pan_joint"/>
-  <xacro:property name="NAME_JOINT_2" value="crane_x7_shoulder_revolute_part_tilt_joint"/>
-  <xacro:property name="NAME_JOINT_3" value="crane_x7_upper_arm_revolute_part_twist_joint"/>
-  <xacro:property name="NAME_JOINT_4" value="crane_x7_upper_arm_revolute_part_rotate_joint"/>
-  <xacro:property name="NAME_JOINT_5" value="crane_x7_lower_arm_fixed_part_joint"/>
-  <xacro:property name="NAME_JOINT_6" value="crane_x7_lower_arm_revolute_part_joint"/>
-  <xacro:property name="NAME_JOINT_7" value="crane_x7_wrist_joint"/>
-  <xacro:property name="NAME_JOINT_COVER_2_L" value="crane_x7_upper_arm_fixed_part_joint_cover_l_joint"/>
-  <xacro:property name="NAME_JOINT_COVER_2_R" value="crane_x7_upper_arm_fixed_part_joint_cover_r_joint"/>
-  <xacro:property name="NAME_JOINT_COVER_4_L" value="crane_x7_lower_arm_fixed_part_joint_cover_l_joint"/>
-  <xacro:property name="NAME_JOINT_COVER_4_R" value="crane_x7_lower_arm_fixed_part_joint_cover_r_joint"/>
-  <xacro:property name="NAME_JOINT_LOGO_SYMBOL_L" value="crane_x7_lower_arm_revolute_part_logo_symbol_l_joint"/>
-  <xacro:property name="NAME_JOINT_LOGO_SYMBOL_R" value="crane_x7_lower_arm_revolute_part_logo_symbol_r_joint"/>
-  <xacro:property name="NAME_JOINT_LOGO_TEXT_L" value="crane_x7_lower_arm_revolute_part_logo_text_l_joint"/>
-  <xacro:property name="NAME_JOINT_LOGO_TEXT_R" value="crane_x7_lower_arm_revolute_part_logo_text_r_joint"/>
-  <xacro:property name="NAME_JOINT_GRIPPER_FINGER_A" value="crane_x7_gripper_finger_a_joint"/>
-  <xacro:property name="NAME_JOINT_GRIPPER_FINGER_B" value="crane_x7_gripper_finger_b_joint"/>
-  <xacro:property name="COLOR_LINK_BASE" value="red"/>
-  <xacro:property name="COLOR_LINK_1" value="white"/>
-  <xacro:property name="COLOR_LINK_COVER_2" value="red"/>
-  <xacro:property name="COLOR_LINK_2" value="white"/>
-  <xacro:property name="COLOR_LINK_3" value="white"/>
-  <xacro:property name="COLOR_LINK_COVER_4" value="red"/>
-  <xacro:property name="COLOR_LINK_4" value="white"/>
-  <xacro:property name="COLOR_LINK_5" value="white"/>
-  <xacro:property name="COLOR_LINK_6" value="white"/>
-  <xacro:property name="COLOR_HAND" value="red"/>
   <xacro:property name="JOINT_VELOCITY_LIMIT" value="4.81710873"/>
   <xacro:property name="JOINT_1_LOWER_LIMIT" value="${radians(-157)}"/>
@@ -105,53 +56,4 @@
   <xacro:crane_x7
     parent="base_link"
-    name_link_mounting_plate="${NAME_LINK_MOUNTING_PLATE}"
-    name_link_base="${NAME_LINK_BASE}"
-    name_link_1="${NAME_LINK_1}"
-    name_link_2="${NAME_LINK_2}"
-    name_link_3="${NAME_LINK_3}"
-    name_link_4="${NAME_LINK_4}"
-    name_link_5="${NAME_LINK_5}"
-    name_link_6="${NAME_LINK_6}"
-    name_link_7="${NAME_LINK_7}"
-    name_link_cover_2_l="${NAME_LINK_COVER_2_L}"
-    name_link_cover_2_r="${NAME_LINK_COVER_2_R}"
-    name_link_cover_4_l="${NAME_LINK_COVER_4_L}"
-    name_link_cover_4_r="${NAME_LINK_COVER_4_R}"
-    name_link_logo_symbol_l="${NAME_LINK_LOGO_SYMBOL_L}"
-    name_link_logo_symbol_r="${NAME_LINK_LOGO_SYMBOL_R}"
-    name_link_logo_text_l="${NAME_LINK_LOGO_TEXT_L}"
-    name_link_logo_text_r="${NAME_LINK_LOGO_TEXT_R}"
-    name_link_gripper_base="${NAME_LINK_GRIPPER_BASE}"
-    name_link_gripper_finger_a="${NAME_LINK_GRIPPER_FINGER_A}"
-    name_link_gripper_finger_b="${NAME_LINK_GRIPPER_FINGER_B}"
-    name_joint_mounting_plate="${NAME_JOINT_MOUNTING_PLATE}"
-    name_joint_base="${NAME_JOINT_BASE}"
-    name_joint_1="${NAME_JOINT_1}"
-    name_joint_2="${NAME_JOINT_2}"
-    name_joint_3="${NAME_JOINT_3}"
-    name_joint_4="${NAME_JOINT_4}"
-    name_joint_5="${NAME_JOINT_5}"
-    name_joint_6="${NAME_JOINT_6}"
-    name_joint_7="${NAME_JOINT_7}"
-    name_joint_cover_2_l="${NAME_JOINT_COVER_2_L}"
-    name_joint_cover_2_r="${NAME_JOINT_COVER_2_R}"
-    name_joint_cover_4_l="${NAME_JOINT_COVER_4_L}"
-    name_joint_cover_4_r="${NAME_JOINT_COVER_4_R}"
-    name_joint_logo_symbol_l="${NAME_JOINT_LOGO_SYMBOL_L}"
-    name_joint_logo_symbol_r="${NAME_JOINT_LOGO_SYMBOL_R}"
-    name_joint_logo_text_l="${NAME_JOINT_LOGO_TEXT_L}"
-    name_joint_logo_text_r="${NAME_JOINT_LOGO_TEXT_R}"
-    name_joint_gripper_finger_a="${NAME_JOINT_GRIPPER_FINGER_A}"
-    name_joint_gripper_finger_b="${NAME_JOINT_GRIPPER_FINGER_B}"
-    color_link_base="${COLOR_LINK_BASE}"
-    color_link_1="${COLOR_LINK_1}"
-    color_link_cover_2="${COLOR_LINK_COVER_2}"
-    color_link_2="${COLOR_LINK_2}"
-    color_link_3="${COLOR_LINK_3}"
-    color_link_cover_4="${COLOR_LINK_COVER_4}"
-    color_link_4="${COLOR_LINK_4}"
-    color_link_5="${COLOR_LINK_5}"
-    color_link_6="${COLOR_LINK_6}"
-    color_hand="${COLOR_HAND}"
     joint_velocity_limit="${JOINT_VELOCITY_LIMIT}"
     joint_1_lower_limit="${JOINT_1_LOWER_LIMIT}"
@@ -177,12 +79,4 @@
     <xacro:crane_x7_ros2_control_settings
       name="crane_x7"
-      name_joint_1="${NAME_JOINT_1}"
-      name_joint_2="${NAME_JOINT_2}"
-      name_joint_3="${NAME_JOINT_3}"
-      name_joint_4="${NAME_JOINT_4}"
-      name_joint_5="${NAME_JOINT_5}"
-      name_joint_6="${NAME_JOINT_6}"
-      name_joint_7="${NAME_JOINT_7}"
-      name_joint_gripper_finger_a="${NAME_JOINT_GRIPPER_FINGER_A}"
       joint_1_lower_limit="${JOINT_1_LOWER_LIMIT}"
       joint_1_upper_limit="${JOINT_1_UPPER_LIMIT}"
@@ -211,23 +105,4 @@
   <xacro:if value="$(arg use_gazebo)">
     <xacro:gazebo_robot_settings
-      name_link_mounting_plate="${NAME_LINK_MOUNTING_PLATE}"
-      name_link_base="${NAME_LINK_BASE}"
-      name_link_1="${NAME_LINK_1}"
-      name_link_2="${NAME_LINK_2}"
-      name_link_3="${NAME_LINK_3}"
-      name_link_4="${NAME_LINK_4}"
-      name_link_5="${NAME_LINK_5}"
-      name_link_6="${NAME_LINK_6}"
-      name_link_cover_2_l="${NAME_LINK_COVER_2_L}"
-      name_link_cover_2_r="${NAME_LINK_COVER_2_R}"
-      name_link_cover_4_l="${NAME_LINK_COVER_4_L}"
-      name_link_cover_4_r="${NAME_LINK_COVER_4_R}"
-      name_link_logo_symbol_l="${NAME_LINK_LOGO_SYMBOL_L}"
-      name_link_logo_symbol_r="${NAME_LINK_LOGO_SYMBOL_R}"
-      name_link_logo_text_l="${NAME_LINK_LOGO_TEXT_L}"
-      name_link_logo_text_r="${NAME_LINK_LOGO_TEXT_R}"
-      name_link_gripper_base="${NAME_LINK_GRIPPER_BASE}"
-      name_link_gripper_finger_a="${NAME_LINK_GRIPPER_FINGER_A}"
-      name_link_gripper_finger_b="${NAME_LINK_GRIPPER_FINGER_B}"
       config_package="$(arg gz_control_config_package)"
       config_file_path="$(arg gz_control_config_file_path)"
@@ -235,13 +110,4 @@
     <xacro:crane_x7_gazebo_ros2_control_settings
       name="crane_x7"
-      name_joint_1="${NAME_JOINT_1}"
-      name_joint_2="${NAME_JOINT_2}"
-      name_joint_3="${NAME_JOINT_3}"
-      name_joint_4="${NAME_JOINT_4}"
-      name_joint_5="${NAME_JOINT_5}"
-      name_joint_6="${NAME_JOINT_6}"
-      name_joint_7="${NAME_JOINT_7}"
-      name_joint_gripper_finger_a="${NAME_JOINT_GRIPPER_FINGER_A}"
-      name_joint_gripper_finger_b="${NAME_JOINT_GRIPPER_FINGER_B}"
       joint_1_lower_limit="${JOINT_1_LOWER_LIMIT}"
       joint_1_upper_limit="${JOINT_1_UPPER_LIMIT}"

File: urdf/crane_x7.xacro (robot description, xacro)
@@ -25,53 +25,4 @@
   <xacro:macro name="crane_x7"
       params="parent
-              name_link_mounting_plate
-              name_link_base
-              name_link_1
-              name_link_2
-              name_link_3
-              name_link_4
-              name_link_5
-              name_link_6
-              name_link_7
-              name_link_cover_2_l
-              name_link_cover_2_r
-              name_link_cover_4_l
-              name_link_cover_4_r
-              name_link_logo_symbol_l
-              name_link_logo_symbol_r
-              name_link_logo_text_l
-              name_link_logo_text_r
-              name_link_gripper_base
-              name_link_gripper_finger_a
-              name_link_gripper_finger_b
-              name_joint_mounting_plate
-              name_joint_base
-              name_joint_1
-              name_joint_2
-              name_joint_3
-              name_joint_4
-              name_joint_5
-              name_joint_6
-              name_joint_7
-              name_joint_cover_2_l
-              name_joint_cover_2_r
-              name_joint_cover_4_l
-              name_joint_cover_4_r
-              name_joint_logo_symbol_l
-              name_joint_logo_symbol_r
-              name_joint_logo_text_l
-              name_joint_logo_text_r
-              name_joint_gripper_finger_a
-              name_joint_gripper_finger_b
-              color_link_base
-              color_link_1
-              color_link_cover_2
-              color_link_2
-              color_link_3
-              color_link_cover_4
-              color_link_4
-              color_link_5
-              color_link_6
-              color_hand
               joint_velocity_limit
               joint_1_lower_limit
@@ -96,54 +47,10 @@
          (Root of the manipulator's TF tree) -->
     <xacro:crane_x7_mounting_plate
-        parent="${parent}"
-        name_link_mounting_plate="${name_link_mounting_plate}"
-        name_joint_mounting_plate="${name_joint_mounting_plate}"
-        color="black">
+      parent="${parent}">
       <xacro:insert_block name="origin"/>
     </xacro:crane_x7_mounting_plate>
     <!-- Arm -->
     <xacro:crane_x7_arm
-        parent="${name_link_mounting_plate}"
-        name_link_base="${name_link_base}"
-        name_link_1="${name_link_1}"
-        name_link_2="${name_link_2}"
-        name_link_3="${name_link_3}"
-        name_link_4="${name_link_4}"
-        name_link_5="${name_link_5}"
-        name_link_6="${name_link_6}"
-        name_link_7="${name_link_7}"
-        name_link_cover_2_l="${name_link_cover_2_l}"
-        name_link_cover_2_r="${name_link_cover_2_r}"
-        name_link_cover_4_l="${name_link_cover_4_l}"
-        name_link_cover_4_r="${name_link_cover_4_r}"
-        name_link_logo_symbol_l="${name_link_logo_symbol_l}"
-        name_link_logo_symbol_r="${name_link_logo_symbol_r}"
-        name_link_logo_text_l="${name_link_logo_text_l}"
-        name_link_logo_text_r="${name_link_logo_text_r}"
-        name_joint_base="${name_joint_base}"
-        name_joint_1="${name_joint_1}"
-        name_joint_2="${name_joint_2}"
-        name_joint_3="${name_joint_3}"
-        name_joint_4="${name_joint_4}"
-        name_joint_5="${name_joint_5}"
-        name_joint_6="${name_joint_6}"
-        name_joint_7="${name_joint_7}"
-        name_joint_cover_2_l="${name_joint_cover_2_l}"
-        name_joint_cover_2_r="${name_joint_cover_2_r}"
-        name_joint_cover_4_l="${name_joint_cover_4_l}"
-        name_joint_cover_4_r="${name_joint_cover_4_r}"
-        name_joint_logo_symbol_l="${name_joint_logo_symbol_l}"
-        name_joint_logo_symbol_r="${name_joint_logo_symbol_r}"
-        name_joint_logo_text_l="${name_joint_logo_text_l}"
-        name_joint_logo_text_r="${name_joint_logo_text_r}"
-        color_link_base="${color_link_base}"
-        color_link_1="${color_link_1}"
-        color_link_cover_2="${color_link_cover_2}"
-        color_link_2="${color_link_2}"
-        color_link_3="${color_link_3}"
-        color_link_cover_4="${color_link_cover_4}"
-        color_link_4="${color_link_4}"
-        color_link_5="${color_link_5}"
-        color_link_6="${color_link_6}"
+      parent="crane_x7_mounting_plate_link"
         joint_velocity_limit="${joint_velocity_limit}"
         joint_1_lower_limit="${joint_1_lower_limit}"
@@ -167,5 +74,5 @@
       <xacro:include filename="$(find realsense2_description)/urdf/_d435.urdf.xacro" />
       <xacro:sensor_d435
-          parent="${name_link_7}"
+          parent="crane_x7_gripper_base_link"
           use_nominal_extrinsics="false"
           add_plug="false"
@@ -176,10 +83,4 @@
     <!-- End effector -->
     <xacro:crane_x7_wide_two_finger_gripper
-        name_link_gripper_base="${name_link_gripper_base}"
-        name_link_gripper_finger_a="${name_link_gripper_finger_a}"
-        name_link_gripper_finger_b="${name_link_gripper_finger_b}"
-        name_joint_gripper_finger_a="${name_joint_gripper_finger_a}"
-        name_joint_gripper_finger_b="${name_joint_gripper_finger_b}"
-        color="${color_hand}"
         joint_velocity_limit="${joint_velocity_limit}"
         joint_hand_lower_limit="${joint_hand_lower_limit}"
