Commit message: Add dummy joint to prevent Joint not found error
[move_group-3] [ERROR] [1692102600.709104192] [moveit_robot_model.robot_model]: Joint 'crane_x7_gripper_finger_b_joint_mimic' not found in model 'crane_x7'

See https://github.com/ros-controls/gazebo_ros2_control/issues/173

File: urdf/crane_x7_wide_two_finger_gripper.xacro (robot description, xacro)
@@ -70,4 +70,12 @@
       </inertial>
     </link>
+    <!--Dummy joint/link to prevent error with mimic joint
+    See https://github.com/ros-controls/gazebo_ros2_control/issues/173
+    -->
+    <joint name="${name_joint_gripper_finger_b}_mimic" type="fixed">
+      <parent link="world" />
+      <child link="dummy_mimic_fix" />
+    </joint>
+    <link name="dummy_mimic_fix"/>
     <joint name="${name_joint_gripper_finger_b}" type="revolute">
       <origin xyz="0.012 0.0 0.024" rpy="0 0 0"/>

Commit message: エラー回避用のdummyジョイントの定義を削除

File: urdf/crane_x7_wide_two_finger_gripper.xacro (robot description, xacro)
@@ -70,12 +70,4 @@
       </inertial>
     </link>
-    <!--Dummy joint/link to prevent error with mimic joint
-    See https://github.com/ros-controls/gazebo_ros2_control/issues/173
-    -->
-    <joint name="${name_joint_gripper_finger_b}_mimic" type="fixed">
-      <parent link="world" />
-      <child link="dummy_mimic_fix" />
-    </joint>
-    <link name="dummy_mimic_fix"/>
     <joint name="${name_joint_gripper_finger_b}" type="revolute">
       <origin xyz="0.012 0.0 0.024" rpy="0 0 0"/>
